File: okabephone.kicad_sch (KiCad schematic)
At the start: 41 parts, among them J1 Micro_SD_Card_Det1, J2 USB_C_Receptacle_USB2.0_16P, M1 Motor_DC, Q1 AO3400A, SW1 SW_Push, SW10 SW_Push, SW11 SW_Push, SW12 SW_Push, SW13 SW_Push, SW14 SW_Push, SW15 SW_Push, SW16 SW_Push, SW17 SW_Push, SW18 SW_Push, SW19 SW_Push, SW2 SW_Push, SW3 SW_Push, SW4 SW_Push, SW5 SW_Push, SW6 SW_Push, SW7 SW_Push, SW8 SW_Push, SW9 SW_Push, U1 MCP23017_ML, U2 ESP32-S3-WROOM-1, U4 SIM7080G, U5 LD1117S33TR_SOT223

Commit message: SD card and stuff?
Parts:
- added C4: 10uF, symbol Device:C
- added C5: 100nF, symbol Device:C
- added R10, R11, R12, R9: 10k, symbol Device:R
Connections:
- net +3.3V: now also R1.1, C4.1, C5.1, R11.1, R12.1
- net GND: now also J1.10 (SHIELD), U1.11 (A0), U1.12 (A1), U1.13 (A2), U1.14 (~{RESET}), C4.2, C5.2, R10.2, R9.2; no longer R1.1
- net SCK: now also R9.1
- net SDA: now also R10.1
- net at SW1.2, SW12.2, SW15.2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: now also U1.26 (GPB1); no longer SW10.1, SW13.1, SW16.1, SW19.1, SW4.1, SW7.1
- net at SW10.2, SW13.2, SW16.2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: now also U1.27 (GPB2)
- net VIBRO_PIN: now reaches R8.1
- net at U1.17 (GPA0): now also SW1.1
- net at U1.18 (GPA1): now also SW2.1, SW3.1, SW4.1
- net at U1.19 (GPA2): now also SW5.1, SW6.1, SW7.1
- net at U1.20 (GPA3): now also SW10.1, SW8.1, SW9.1
- net at U1.21 (GPA4): now also SW11.1, SW12.1, SW13.1
- net at U1.22 (GPA5): now also SW14.1, SW15.1, SW16.1
- net at U1.23 (GPA6): now also SW17.1, SW18.1, SW19.1
- net at U1.25 (GPB0): now also SW11.2, SW14.2, SW17.2, SW2.2, SW5.2, SW8.2
- net SD_CS: now reaches R1.2
- net SD_CS: now also J1.2 (DAT3/CD); no longer J1.10 (SHIELD)
- net SD_MOSI: now reaches J1.3 (CMD)
- net SD_MOSI: now also R11.2
- net SD_SCK: now reaches J1.5 (CLK)
- net SD_MISO: now reaches J1.7 (DAT0)
- net SD_MISO: now also R12.2
- net SD_DET: now reaches J1.9 (DET)
- no-connect marks 3 -> 11
Other:
- moved on the sheet: D1, F1, SW1, SW10, SW11, SW12, SW13, SW14, SW15, SW16, SW17, SW18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

Commit message: t
Parts:
- removed C1: 10uF, symbol Device:C
- removed C2: 22uF, symbol Device:C
- removed D1: D_TVS, symbol Device:D_TVS
- removed F1: Polyfuse, symbol Device:Polyfuse
- removed J2: USB_C_Receptacle_USB2.0_16P, symbol Connector:USB_C_Receptacle_USB2.0_16P
- removed R4, R5: 5.1k, symbol Device:R
- removed R6, R7: 100k, symbol Device:R
- removed U4: SIM7080G, SIM7080G:XCVR_SIM7080G, symbol SIM7080G:SIM7080G
- removed U5: LD1117S33TR_SOT223, Package_TO_SOT_SMD:SOT-223-3_TabPin2, symbol Regulator_Linear:LD1117S33TR_SOT223
- added C6: 100nF, symbol Device:C
- added RX0-TP, TX0-TP: TestPoint, symbol Connector:TestPoint
- added U6: PCF8563T, Package_SO:SOIC-8_3.9x4.9mm_P1.27mm, symbol Timer_RTC:PCF8563T
- added Y1: 32.768kHz, Crystal:Crystal_SMD_3215-2Pin_3.2x1.5mm, symbol Device:Crystal
Connections:
- net +3.3V: now also R10.2, R9.2
- net +BATT: now also C6.1, U6.8 (VDD); no longer C3.1, M1.1 (+)
- net GND: now also C6.2, U6.4 (VSS); no longer R10.2, R9.2
- net SCK: now also U6.6 (SCL)
- net SDA: now also U6.5 (SDA)
- net at U2.36 (RXD0): now also RX0-TP.1
- net at U2.37 (TXD0): now also TX0-TP.1
- new net: U6.1 (OSCI), Y1.2
- new net: U6.2 (OSCO), Y1.1
- new net RTC_ALARM_INT: U6.3 (~{INT})
- new net VBAT: C3.1, M1.1 (+)
- no-connect marks 11 -> 12
Other:
- added sheet CELLULAR (cellular.kicad_sch)
- added sheet POWER (power.kicad_sch)
- company: (none) -> Nergon
- title: (none) -> Okabe_Phone
- moved on the sheet: C3, C4, C5, D2, J1, M1, Q1, R1, R10, R11, R12, R2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

Commit message: power
Other:
- moved on the sheet: R10, R9
Changed lines of the file:
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@@
 	)
 	(junction
-		(at 33.02 95.25)
+		(at 210.82 27.94)
 		(diameter 0)
 		(color 0 0 0 0)
@@
 	(wire
 		(pts
-			(xy 33.02 93.98) (xy 35.56 93.98)
+			(xy 210.82 26.67) (xy 213.36 26.67)
 		)
 		(stroke
@@
 	(wire
 		(pts
-			(xy 44.45 93.98) (xy 43.18 93.98)
+			(xy 222.25 26.67) (xy 220.98 26.67)
 		)
 		(stroke
@@
 	(wire
 		(pts
-			(xy 44.45 96.52) (xy 43.18 96.52)
+			(xy 222.25 29.21) (xy 220.98 29.21)
 		)
 		(stroke
@@
 	(wire
 		(pts
-			(xy 33.02 93.98) (xy 33.02 95.25)
+			(xy 210.82 26.67) (xy 210.82 27.94)
 		)
 		(stroke
@@
 	(wire
 		(pts
-			(xy 33.02 96.52) (xy 35.56 96.52)
+			(xy 210.82 29.21) (xy 213.36 29.21)
 		)
 		(stroke
@@
 	(wire
 		(pts
-			(xy 33.02 96.52) (xy 33.02 95.25)
+			(xy 210.82 29.21) (xy 210.82 27.94)
 		)
 		(stroke
@@
 	)
 	(label "I2C pullup"
-		(at 31.75 90.17 0)
+		(at 209.55 22.86 0)
 		(effects
 			(font
@@
 	(global_label "SDA"
 		(shape bidirectional)
-		(at 44.45 96.52 0)
+		(at 222.25 29.21 0)
 		(fields_autoplaced yes)
 		(effects
@@
 		)
 		(property "Intersheetrefs" "${INTERSHEET_REFS}"
-			(at 52.1146 96.52 0)
+			(at 229.9146 29.21 0)
 			(effects
 				(font
@@
 	(global_label "SCK"
 		(shape bidirectional)
-		(at 44.45 93.98 0)
+		(at 222.25 26.67 0)
 		(fields_autoplaced yes)
 		(effects
@@
 		)
 		(property "Intersheetrefs" "${INTERSHEET_REFS}"
-			(at 52.296 93.98 0)
+			(at 230.096 26.67 0)
 			(effects
 				(font
@@
 	(symbol
 		(lib_id "Device:R")
-		(at 39.37 93.98 270)
+		(at 217.17 26.67 270)
 		(unit 1)
 		(exclude_from_sim no)
@@
 		(dnp no)
 		(property "Reference" "R9"
-			(at 37.846 91.694 90)
+			(at 215.646 24.384 90)
 			(effects
 				(font
@@
 		)
 		(property "Value" "10k"
-			(at 37.084 93.98 90)
+			(at 214.884 26.67 90)
 			(effects
 				(font
@@
 		)
 		(property "Footprint" ""
-			(at 39.37 92.202 90)
+			(at 217.17 24.892 90)
 			(effects
 				(font
@@
 		)
 		(property "Datasheet" "~"
-			(at 39.37 93.98 0)
+			(at 217.17 26.67 0)
 			(effects
 				(font
@@
 		)
 		(property "Description" "Resistor"
-			(at 39.37 93.98 0)
+			(at 217.17 26.67 0)
 			(effects
 				(font
@@
 	(symbol
 		(lib_id "power:+3.3V")
-		(at 33.02 95.25 90)
+		(at 210.82 27.94 90)
 		(unit 1)
 		(exclude_from_sim no)
@@
 		(dnp no)
 		(property "Reference" "#PWR06"
-			(at 36.83 95.25 0)
+			(at 214.63 27.94 0)
 			(effects
 				(font
@@
 		)
 		(property "Value" "+3.3V"
-			(at 27.94 95.25 0)
+			(at 205.74 27.94 0)
 			(effects
 				(font
@@
 		)
 		(property "Footprint" ""
-			(at 33.02 95.25 0)
+			(at 210.82 27.94 0)
 			(effects
 				(font
@@
 		)
 		(property "Datasheet" ""
-			(at 33.02 95.25 0)
+			(at 210.82 27.94 0)
 			(effects
 				(font
@@
 		)
 		(property "Description" "Power symbol creates a global label with name \"+3.3V\""
-			(at 33.02 95.25 0)
+			(at 210.82 27.94 0)
 			(effects
 				(font
@@
 		(on_board yes)
 		(dnp no)
-		(fields_autoplaced yes)
 		(property "Reference" "#PWR07"
 			(at 46.99 83.82 0)
@@
 	(symbol
 		(lib_id "Device:R")
-		(at 39.37 96.52 270)
+		(at 217.17 29.21 270)
 		(unit 1)
 		(exclude_from_sim no)
@@
 		(dnp no)
 		(property "Reference" "R10"
-			(at 37.846 99.06 90)
+			(at 215.646 31.75 90)
 			(effects
 				(font
@@
 		)
 		(property "Value" "10k"
-			(at 37.084 96.52 90)
+			(at 214.884 29.21 90)
 			(effects
 				(font
@@
 		)
 		(property "Footprint" ""
-			(at 39.37 94.742 90)
+			(at 217.17 27.432 90)
 			(effects
 				(font
@@
 		)
 		(property "Datasheet" "~"
-			(at 39.37 96.52 0)
+			(at 217.17 29.21 0)
 			(effects
 				(font
@@
 		)
 		(property "Description" "Resistor"
-			(at 39.37 96.52 0)
+			(at 217.17 29.21 0)
 			(effects
 				(font

Commit message: spi joke
Connections:
- net SD_MISO is gone; now on net SCR_MISO: J1.7 (DAT0), R12.2
- net SD_MOSI is gone; now on net SCR_MOSI: J1.3 (CMD), R11.2
- net SD_SCK is gone; now on net SCR_SCK: J1.5 (CLK)
- net SCK: now also U2.18 (IO10)
- net SDA: now also U2.17 (IO9)
- net SD_CS: now also U2.39 (IO1)
- net SD_DET: now also U2.6 (IO6)
- net VIBRO_PIN: now also U2.12 (IO8)
- net SIM_RX: now reaches U2.10 (IO17)
- net SIM_TX: now reaches U2.11 (IO18)
- net SCR_SCK: now reaches U2.15 (IO3)
- net BOOT46: now reaches U2.16 (IO46)
- net CHG_PIN: now reaches U2.19 (IO11)
- net PWR_HOLD: now reaches U2.20 (IO12)
- net PWRBTN_DETECT: now reaches U2.21 (IO13)
- net SIM_RI: now reaches U2.23 (IO21)
- net BOOT0: now reaches U2.27 (IO0)
- net SCR_MOSI: now reaches U2.38 (IO2)
- net SCR_MISO: now reaches U2.4 (IO4)
- net SCR_CS: now reaches U2.5 (IO5)
- net SCR_PWM: now reaches U2.7 (IO7)

Commit message: buck converter
Parts:
- added C10, C11: 100nF, symbol Device:C
- added C12: 10uF, symbol Device:C
- added R25: 10k, symbol Device:R
- added SW21: SW_Push, symbol Switch:SW_Push
- renumbered RX0-TP to RX0-TP1, TX0-TP to TX0-TP1
Connections:
- net +3.3V: now also C11.1, C12.1, R25.1
- net GND: now also C10.1, C11.2, C12.2, SW21.1
- net SIM_RI: now also U2.9 (IO16); no longer U2.23 (IO21)
- net SIM_RX: now also U2.22 (IO14); no longer U2.10 (IO17)
- net SIM_TX: now also U2.8 (IO15); no longer U2.11 (IO18)
- net at U2.3 (EN): now also C10.2, R25.2, SW21.2
Other:
- moved on the sheet: C3, C4, C5, D2, M1, Q1, R10, R2, R3, R8, R9, RX0-TP1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

Commit message: eee:
Parts:
- added F2, F3: Polyfuse, symbol Device:Polyfuse
- added J6: SFH11-PBPC-D10-RA-BK, CONN20_D10-RA-BK_SUL, symbol 20PIN Connector:SFH11-PBPC-D10-RA-BK
Connections:
- net +3.3V: now also F2.1
- net BOOT0: now also J6.16
- net BOOT46: now also J6.15
- net GND: now also J6.17, J6.18, J6.19, J6.20
- net RTC_ALARM_INT: now also U2.35 (IO42)
- net SCK: now also J6.2
- net SDA: now also J6.1
- net AUD_RESET: now reaches U2.10 (IO17)
- net AUD_DIN: now reaches U2.11 (IO18)
- net AUD_DOUT: now reaches U2.23 (IO21)
- net IO47: now reaches U2.24 (IO47)
- net IO47: now also J6.9
- net IO48: now reaches U2.25 (IO48)
- net IO48: now also J6.8
- net MCP_INT_B: now reaches U2.26 (IO45)
- net MCP_INT_B: now also U1.15 (INTB)
- net OUT_IO_35: now reaches U2.28 (IO35)
- net OUT_IO_35: now also J6.7
- net OUT_IO_36: now reaches U2.29 (IO36)
- net OUT_IO_36: now also J6.6
- net OUT_IO_37: now reaches U2.30 (IO37)
- net OUT_IO_37: now also J6.5
- net AUD_BCLK: now reaches U2.31 (IO38)
- net AUD_WCLK: now reaches U2.32 (IO39)
- net AUD_MCLK: now reaches U2.33 (IO40)
- net AUD_GPIO: now reaches U2.34 (IO41)
- net OUT_RXD: now reaches RX0-TP1.1, U2.36 (RXD0)
- net OUT_RXD: now also J6.3
- net OUT_TXD: now reaches TX0-TP1.1, U2.37 (TXD0)
- net OUT_TXD: now also J6.4
- net SCR_MISO renamed OUT_MISO
- net OUT_MISO: now also J6.10
- net SCR_MOSI renamed OUT_MOSI
- net OUT_MOSI: now also J6.12
- net SCR_SCK renamed OUT_SCK
- net OUT_SCK: now also J6.11
- new net: F2.2, J6.13
- new net: F3.2, J6.14
- new net +VSW: F3.1
- no-connect marks 12 -> 9
Other:
- added sheet AUDIO (AUDIO.kicad_sch)
- moved on the sheet: C10, C3, D2, M1, Q1, R25, R8, RX0-TP1, SW21, TX0-TP1

Commit message: :)
Parts:
- J6: footprint CONN20_D10-RA-BK_SUL -> connector:CONN20_D10-RA-BK_SUL
- U2: footprint RF_Module:ESP32-S3-WROOM-1 -> RF_Module:ESP32-S3-WROOM-1U
Connections:
- net GND: no longer J6.17
- net SCK: now also J6.14; no longer J6.2
- net SDA: now also J6.13; no longer J6.1
- net ESP_EN: now reaches C10.2, R25.2, SW21.2, U2.3 (EN)
- net ESP_EN: now also J6.17
- net at F2.2: now also J6.1; no longer J6.13
- net at F3.2: now also J6.2; no longer J6.14
Other:
- moved on the sheet: F2, F3

Commit message: mblya
Parts:
- removed C10, C11, C5, C6: 100nF, symbol Device:C
- removed C12, C4: 10uF, symbol Device:C
- removed C3: 1uF, symbol Device:C
- removed D2: SS14, Diode_SMD:D_SMA, symbol Diode:SS14
- removed F2, F3: Polyfuse, symbol Device:Polyfuse
- removed J6: SFH11-PBPC-D10-RA-BK, connector:CONN20_D10-RA-BK_SUL, symbol 20PIN Connector:SFH11-PBPC-D10-RA-BK
- removed R10, R11, R12, R9: 10k, symbol Device:R
- removed R2, R3: 22, symbol Device:R
- removed R8: 220, symbol Device:R
- removed RX0-TP1, TX0-TP1: TestPoint, symbol Connector:TestPoint
- removed SW1, SW10, SW11, SW12, SW13, SW14, SW15, SW16, SW17, SW18, SW19, SW2, SW21, SW3, SW4, SW5, SW6, SW7, SW8, SW9: SW_Push, symbol Switch:SW_Push
- removed U6: PCF8563T, Package_SO:SOIC-8_3.9x4.9mm_P1.27mm, symbol Timer_RTC:PCF8563T
- removed Y1: 32.768kHz, Crystal:Crystal_SMD_3215-2Pin_3.2x1.5mm, symbol Device:Crystal
- added C25, C27, C29, C31, C33: 10uF, symbol Device:C
- added C26, C28, C30, C32, C34: 100nF, symbol Device:C
- added D6: 1N5819WS, Diode_SMD:D_SOD-323, symbol Diode:1N5819WS
- added R15, R16: 22, symbol Device:R
- added R17, R23: 10k, symbol Device:R
- added R24: 1k, symbol Device:R
- added R26: 6.8, symbol Device:R
- added RXD, TXD: TestPoint, symbol Connector:TestPoint
- added SW1, SW10, SW11, SW12, SW13, SW14, SW15, SW16, SW17, SW18, SW19, SW2, SW3, SW4, SW5, SW6, SW7, SW8, SW9, SW_BOOT, SW_RST: SW_MEC_5E, symbol Switch:SW_MEC_5E
- added TP8: 3.3V, symbol Connector:TestPoint
- added TP9: GND, symbol Connector:TestPoint
- added U8: PCF8563T, Package_SO:SOIC-8_3.9x4.9mm_P1.27mm, symbol Timer_RTC:PCF8563T
- R25: value 10k -> 200k
- U2: footprint RF_Module:ESP32-S3-WROOM-1U -> RF_Module:ESP32-S3-WROOM-1
Connections:
- net +3.3V: now also U1.14 (~{RESET}), C25.2, C26.2, C27.2, C28.2, C29.2, C30.2, C31.2, C32.2, R17.1, R23.2, R26.1, TP8.1; no longer R25.1
- net +VSW: now also C33.2, C34.2, U8.8 (VDD)
- net GND: now also R25.1, C25.1, C26.1, C27.1, C28.1, C29.1, C30.1, C31.1, C32.1, C33.1, C34.1, SW_BOOT.3 (K), SW_BOOT.4 (A), SW_RST.3 (K), SW_RST.4 (A), TP9.1, U8.4 (VSS); no longer U1.14 (~{RESET})
- net SCK: now also R23.1, U8.6 (SCL); no longer U2.18 (IO10)
- net SCR_CS: no longer U2.5 (IO5)
- net SDA: now also R17.2, U8.5 (SDA); no longer U2.17 (IO9)
- net USB_DN: now also R16.2
- net USB_DP: now also R15.2
- net at M1.2 (-): now also Q1.3 (D), D6.2 (A)
- net at U1.19 (GPA2): now also SW14.1
- net at U1.27 (GPB2): now also SW19.3 (K)
- net at U2.13 (USB_D-): now also R16.1
- net at U2.14 (USB_D+): now also R15.1
- net at U1.21 (GPA4): now also SW8.1
- net at Q1.1 (G): now also R24.2
- net at U1.25 (GPB0): now also SW15.3 (K)
- net at U1.26 (GPB1): now also SW17.3 (K)
- net at U1.18 (GPA1): now also SW15.1
- net at U1.20 (GPA3): now also SW9.1
- net at U1.22 (GPA5): now also SW5.1
- net at U1.23 (GPA6): now also SW2.1
- net at U1.24 (GPA7): now also SW1.1
- net AUD_BCLK: no longer names the net of U2.31 (IO38)
- net AUD_DIN: no longer names the net of U2.11 (IO18)
- net AUD_DOUT: no longer names the net of U2.23 (IO21)
- net AUD_GPIO: no longer names the net of U2.34 (IO41)
- net AUD_MCLK: no longer names the net of U2.33 (IO40)
- net AUD_RESET: no longer names the net of U2.10 (IO17)
- net AUD_WCLK: no longer names the net of U2.32 (IO39)
- net BOOT0 renamed SOC_BOOT
- net SOC_BOOT: now also SW_BOOT.2
- net BOOT46: no longer names the net of U2.16 (IO46)
- net CHG_PIN: no longer names the net of U2.19 (IO11)
- net ESP_EN renamed SOC_EN
- net SOC_EN: now also R1.2, SW_RST.1; no longer R25.2
- net IO47: no longer names the net of U2.24 (IO47)
- net IO48: no longer names the net of U2.25 (IO48)
- net MCP_INT_B: no longer names the net of U2.26 (IO45)
- net MCP_INT_B: no longer U1.15 (INTB)
- net OUT_IO_35: no longer names the net of U2.28 (IO35)
- net OUT_IO_36: no longer names the net of U2.29 (IO36)
- net OUT_IO_37: no longer names the net of U2.30 (IO37)
- net OUT_MISO: no longer names the net of U2.4 (IO4)
- net OUT_MISO: no longer J1.7 (DAT0)
- net OUT_MOSI: no longer names the net of U2.38 (IO2)
- net OUT_MOSI: no longer J1.3 (CMD)
- net OUT_RXD: no longer names the net of U2.36 (RXD0)
- net OUT_RXD: now also RXD.1
- net OUT_SCK: no longer names the net of U2.15 (IO3)
- net OUT_SCK: no longer J1.5 (CLK)
- net OUT_TXD: no longer names the net of U2.37 (TXD0)
- net OUT_TXD: now also TXD.1
- net PWRBTN_DETECT: no longer names the net of U2.21 (IO13)
- net PWR_HOLD: no longer names the net of U2.20 (IO12)
- net RTC_ALARM_INT: no longer names the net of U2.35 (IO42)
- net SCR_PWM: no longer names the net of U2.7 (IO7)
- removed net SD_CS: J1.2 (DAT3/CD), R1.2, U2.39 (IO1)
- net SD_DET: no longer names the net of U2.6 (IO6)
- net SD_DET: no longer J1.9 (DET)
- net SIM_RI: no longer names the net of U2.9 (IO16)
- net SIM_RX: no longer names the net of U2.22 (IO14)
- net SIM_TX: no longer names the net of U2.8 (IO15)
- net VBAT: no longer names the net of M1.1 (+)
- net VBAT: now also D6.1 (K), R26.2
- net VIBRO_PIN: no longer names the net of U2.12 (IO8)
- new net: SW5.2, SW6.1
- new net: SW5.3 (K), SW8.4 (A)
- new net: SW2.3 (K), SW5.4 (A)
- new net: SW10.1, SW8.2
- new net: SW8.3 (K), SW9.4 (A)
- new net: SW15.2, SW17.1
- new net: SW14.3 (K), SW15.4 (A)
- new net: SW3.2, SW4.1
- new net: SW4.3 (K), SW7.4 (A)
- new net: SW1.3 (K), SW3.4 (A)
- new net: SW10.2, SW12.1
- new net: SW12.3 (K), SW13.4 (A)
- new net: SW12.4 (A), SW7.3 (K)
- new net: SW14.2, SW16.1
- new net: SW16.2, SW18.1
- new net: SW16.3 (K), SW17.4 (A)
- new net: SW11.3 (K), SW16.4 (A)
- new net: SW11.2, SW13.1
- new net: SW13.3 (K), SW18.4 (A)
- new net: SW6.2, SW7.1
- new net: SW11.1, SW9.2
- new net: SW10.3 (K), SW11.4 (A)
- new net: SW2.2, SW3.1
- new net: SW14.4 (A), SW9.3 (K)
- new net: SW3.3 (K), SW6.4 (A)
- new net: SW10.4 (A), SW6.3 (K)
- new net: SW17.2, SW19.1
- new net: SW18.3 (K), SW19.4 (A)
- new net INT_ALARM: U8.3 (~{INT})
- new net MISO: J1.7 (DAT0)
- new net MOSI: J1.3 (CMD)
- new net SPI_CLOCK: J1.5 (CLK)
- new net TF_CS: J1.2 (DAT3/CD)
- new net VIB_CTRL: R24.1, R25.2
- no-connect marks 9 -> 10
Other:
- company: Nergon -> (none)
- title: Okabe_Phone -> (none)
- moved on the sheet: J1, M1, U1, U2
