File: cellular.kicad_sch (KiCad schematic)
At the start: 6 parts, among them Q2 BC547, U3 A7672SA__LASE_, U4 LoRa-E5

Commit message: power
Changed lines of the file:
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@@
 		)
 	)
-	(label "LoRa Chip"
+	(label "LoRa Module"
 		(at 247.65 81.28 0)
 		(effects

Commit message: spi joke
Parts:
- removed U4: LoRa-E5, LoRa-E5:LoRa-E5, symbol LoRa-E5:LoRa-E5
- added C7: 1nF, symbol Device:C
- added J4: SIM_Card, symbol Connector:SIM_Card
- added R18: 680k, symbol Device:R
- added R19: 470k, symbol Device:R
- added R20, R21, R22: R, symbol Device:R
- added TP1: S_LOGR, symbol Connector:TestPoint
- added TP2: S_LOGT, symbol Connector:TestPoint
- added TP3: S_USBP, symbol Connector:TestPoint
- added TP4: S_USBM, symbol Connector:TestPoint
- added TP5: S_VBUS, symbol Connector:TestPoint
- added TP6: S_BOOT, symbol Connector:TestPoint
Connections:
- net GND: now also C7.2, R19.2
- net at U3.22 (UART_LOG_RX): now also TP1.1
- net at U3.23 (UART_LOG_TX): now also TP2.1
- net at U3.24 (VBUS): now also TP5.1
- net at U3.27 (USB_DP): now also TP3.1
- net at U3.28 (USB_DM): now also TP4.1
- net sim1_dat: now reaches U3.31 (USIM1_DATA)
- net sim1_clk: now reaches U3.32 (USIM1_CLK)
- net sim1_rst: now reaches U3.33 (USIM1_RST)
- net at U3.51 (VBAT_ADC): now also C7.1, R18.2, R19.1
- net at U3.6 (USB_BOOT): now also TP6.1
- new net +BATT: R18.1
- no-connect marks 65 -> 53

Commit message: buck converter
Parts:
- R20, R21, R22: value R -> 22
Connections:
- net GND: now also J4.5 (GND), U3.17 (GND_1), U3.18 (GND_1), U3.2 (GND_1), U3.29 (GND_1), U3.39 (GND_1), U3.45 (GND_1), U3.46 (GND_1), U3.54 (GND_1), U3.58 (GND_1), U3.59 (GND_1), U3.61 (GND_1), U3.62 (GND_1), U3.63 (GND_1), U3.64 (GND_1), U3.65 (GND_1), U3.69 (GND_2), U3.70 (GND_2), U3.71 (GND_2), U3.72 (GND_2), U3.73 (GND_2), U3.74 (GND_2), U3.75 (GND_2), U3.76 (GND_2), U3.77 (GND_2), U3.78 (GND_2), U3.79 (GND_2), U3.80 (GND_2), U3.81 (GND_2), U3.82 (GND_2), U3.83 (GND_2), U3.84 (GND_3), U3.85 (GND_3), U3.86 (GND_3), U3.87 (GND_3), U3.88 (GND_3), U3.89 (GND_3), U3.91 (GND_3), U3.92 (GND_3), U3.94 (GND_3)
- net sim1_clk: now also R21.1
- net sim1_dat: now also R20.1
- net sim1_rst: now also R22.1
- net sim1_vdd: now reaches J4.1 (VCC)
- net sim1_vdd: now also U3.30 (USIM1_VDD)
- net at J4.2 (RST): now also R22.2
- net at J4.3 (CLK): now also R21.2
- net at J4.7 (I/O): now also R20.2
- new net: U3.113 (NC), U3.114 (NC), U3.115 (NC)
- new net VBAT: U3.55 (VBAT), U3.56 (VBAT), U3.57 (VBAT)

Commit message: eee:
Parts:
- added C14, C15, C16: 22pF, symbol Device:C
- added C17: 100nF, symbol Device:C
- added C18: 33pF, symbol Device:C
- added unit 1 of U3
- added U5: SMF15CT1G, SMF15CT1G:SOT65P210X110-6N, symbol SMF15CT1G:SMF15CT1G
Connections:
- net GND: now also C14.2, C15.2, C16.2, C17.2, C18.2, U5.2 (A); no longer U3.41 (EAR_N), U3.43 (MIC_N)
- net sim1_clk: now also U3.32 (USIM1_CLK); no longer U3.32 (USIM1_CLK)
- net sim1_dat: now also U3.31 (USIM1_DATA); no longer U3.31 (USIM1_DATA)
- net sim1_rst: now also U3.33 (USIM1_RST); no longer U3.33 (USIM1_RST)
- net sim1_vdd: now also C17.1, C18.1, U5.1 (K_1)
- net at TP6.1: now also U3.6 (USB_BOOT); no longer U3.6 (USB_BOOT)
- net at TP1.1: now also U3.22 (UART_LOG_RX); no longer U3.22 (UART_LOG_RX)
- net at C7.1, R18.2, R19.1: now also U3.51 (VBAT_ADC); no longer U3.51 (VBAT_ADC)
- net at TP3.1: now also U3.27 (USB_DP); no longer U3.27 (USB_DP)
- net at TP2.1: now also U3.23 (UART_LOG_TX); no longer U3.23 (UART_LOG_TX)
- net at J4.2 (RST), R22.2: now also C16.1, U5.3 (K_2)
- net at J4.3 (CLK), R21.2: now also C15.1, U5.4 (K_3)
- net at J4.7 (I/O), R20.2: now also C14.1, U5.5 (K_4)
- net at TP5.1: now also U3.24 (VBUS); no longer U3.24 (VBUS)
- net at D3.2 (A2), Q2.1 (C): now also U3.1 (~{PWRKEY}); no longer U3.1 (~{PWRKEY})
- net at TP4.1: now also U3.28 (USB_DM); no longer U3.28 (USB_DM)
- net +1V8: now reaches U3.15 (VDD_1V8)
- net VBAT renamed +VSW
- new net SIM_EAR_N: U3.41 (EAR_N)
- new net SIM_EAR_P: U3.40 (EAR_P)
- no-connect marks 53 -> 54
Other:
- moved on the sheet: R20, R21, R22, U3B

Commit message: :)
Parts:
- removed Q2: BC547, Package_TO_SOT_THT:TO-92_Inline, symbol Transistor_BJT:BC547
- added Q2: BC847, Package_TO_SOT_SMD:SOT-23, symbol Transistor_BJT:BC847
Connections:
- net GND: now also Q2.2 (E)
- net at R13.2, R14.2: now also Q2.1 (B)
- net at D3.2 (A2), U3.1 (~{PWRKEY}): now also Q2.3 (C)
Changed lines of the file:
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@@
+	)
+	(symbol
+		(lib_id "Transistor_BJT:BC847")
+		(at 48.26 33.02 0)
+		(unit 1)
+		(exclude_from_sim no)
+		(in_bom yes)
+		(on_board yes)
+		(dnp no)
+		(fields_autoplaced yes)
+		(property "Reference" "Q2"
+			(at 53.34 31.7499 0)
+			(effects
+				(font
+					(size 1.27 1.27)
+				)
+				(justify left)
+			)
+		)
+		(property "Value" "BC847"
+			(at 53.34 34.2899 0)
+			(effects
+				(font
+					(size 1.27 1.27)
+				)
+				(justify left)
+			)
+		)
+		(property "Footprint" "Package_TO_SOT_SMD:SOT-23"
+			(at 53.34 34.925 0)
+			(effects
+				(font
+					(size 1.27 1.27)
+					(italic yes)
+				)
+				(justify left)
+				(hide yes)
+			)
+		)
+		(property "Datasheet" "http://www.infineon.com/dgdl/Infineon-BC847SERIES_BC848SERIES_BC849SERIES_BC850SERIES-DS-v01_01-en.pdf?fileId=db3a304314dca389011541d4630a1657"
+			(at 48.26 33.02 0)
+			(effects
+				(font
+					(size 1.27 1.27)
+				)
+				(justify left)
+				(hide yes)
+			)
+		)
+		(property "Description" "0.1A Ic, 45V Vce, NPN Transistor, SOT-23"
+			(at 48.26 33.02 0)
+			(effects
+				(font
+					(size 1.27 1.27)
+				)
+				(hide yes)
+			)
+		)
+		(property "Sim.Device" "NPN"
+			(at 48.26 33.02 0)
+			(effects
+				(font
+					(size 1.27 1.27)
+				)
+				(hide yes)
+			)
+		)
+		(property "Sim.Pins" "1=B 2=E 3=C"
+			(at 48.26 33.02 0)
+			(effects
+				(font
+					(size 1.27 1.27)
+				)
+				(hide yes)
+			)
+		)
+		(pin "2"
+		)
+		(pin "3"
+		)
+		(pin "1"
+		)
+		(instances
+			(project ""
+				(path "/e9d3405d-3536-4ebc-8db6-e75908125fac/8fc5f1cb-84ec-4bac-b8ef-bc0461400e20"
+					(reference "Q2")
+					(unit 1)
+				)
+			)
+		)
 	)
 	(symbol
@@
 					(unit 1)
 				)
-			)
-		)
-	)
-	(symbol
-		(lib_id "Transistor_BJT:BC547")
-		(at 48.26 33.02 0)
-		(unit 1)
-		(exclude_from_sim no)
-		(in_bom yes)
-		(on_board yes)
-		(dnp no)
-		(fields_autoplaced yes)
-		(property "Reference" "Q2"
-			(at 53.34 31.7499 0)
-			(effects
-				(font
-					(size 1.27 1.27)
-				)
-				(justify left)
-			)
-		)
-		(property "Value" "BC547"
-			(at 53.34 34.2899 0)
-			(effects
-				(font
-					(size 1.27 1.27)
-				)
-				(justify left)
-			)
-		)
-		(property "Footprint" "Package_TO_SOT_THT:TO-92_Inline"
-			(at 53.34 34.925 0)
-			(effects
-				(font
-					(size 1.27 1.27)
-					(italic yes)
-				)
-				(justify left)
-				(hide yes)
-			)
-		)
-		(property "Datasheet" "https://www.onsemi.com/pub/Collateral/BC550-D.pdf"
-			(at 48.26 33.02 0)
-			(effects
-				(font
-					(size 1.27 1.27)
-				)
-				(justify left)
-				(hide yes)
-			)
-		)
-		(property "Description" "0.1A Ic, 45V Vce, Small Signal NPN Transistor, TO-92"
-			(at 48.26 33.02 0)
-			(effects
-				(font
-					(size 1.27 1.27)
-				)
-				(hide yes)
-			)
-		)
-		(property "Sim.Device" "NPN"
-			(at 48.26 33.02 0)
-			(effects
-				(font
-					(size 1.27 1.27)
-				)
-				(hide yes)
-			)
-		)
-		(property "Sim.Pins" "1=C 2=B 3=E"
-			(at 48.26 33.02 0)
-			(effects
-				(font
-					(size 1.27 1.27)
-				)
-				(hide yes)
-			)
-		)
-		(pin "2"
-		)
-		(pin "1"
-		)
-		(pin "3"
-		)
-		(instances
-			(project "okabephone"
-				(path "/e9d3405d-3536-4ebc-8db6-e75908125fac/8fc5f1cb-84ec-4bac-b8ef-bc0461400e20"
-					(reference "Q2")
-					(unit 1)
-				)

Commit message: SCHEMATIC
Parts:
- removed TP6: S_BOOT, symbol Connector:TestPoint
- added 1V8_SIM, PWRKEY, USB_BOOT, VBAT_ADC, VBAT_SIM, VBAT_SIM1, VBAT_SIM2: SolderJumper_2_Open, Jumper:SolderJumper-2_P1.3mm_Open_Pad1.0x1.5mm, symbol Jumper:SolderJumper_2_Open
- added C40, C41, C42: 22pF, symbol Device:C
- added C43, C45, C46: 100nF, symbol Device:C
- added C44: 33pF, symbol Device:C
- added EAR_N, EAR_P, MIC_N, MIC_P: TestPoint, symbol Connector:TestPoint
- added J2: SIM_Card, symbol Connector:SIM_Card
- added R33: 10k, symbol Device:R
- added R34, R35, R36: 22, symbol Device:R
- added U10: SMF15CT1G, SMF15CT1G:SOT65P210X110-6N, symbol SMF15CT1G:SMF15CT1G
- added U11: SN74AXC4T245PWR, TSSOP16_PW_TEX, symbol SN74AXC4T245PWR:SN74AXC4T245PWR
- added U9: ~, symbol A7676E:A7676E
- C7: value 1nF -> 1uF
Connections:
- net +1V8: now also 1V8_SIM.2 (B), C45.1, U11.1 (VCCA), U11.2 (1DIR)
- net +BATT: now also VBAT_SIM.2 (B), VBAT_SIM1.2 (B), VBAT_SIM2.2 (B)
- net GND: now also C40.2, C41.2, C42.2, C43.2, C44.2, C45.2, C46.2, J2.5 (GND), R33.2, U10.2 (A), U11.14 (2*OE), U11.15 (1*OE), U11.3 (2DIR), U11.8 (GND), U11.9 (GND), U9.17 (GND), U9.18 (GND), U9.2 (GND), U9.29 (GND), U9.39 (GND), U9.45 (GND), U9.46 (GND), U9.54 (GND), U9.58 (GND), U9.59 (GND), U9.61 (GND), U9.62 (GND), U9.63 (GND), U9.64 (GND), U9.65 (GND), U9.69 (GND), U9.70 (GND), U9.71 (GND), U9.72 (GND), U9.73 (GND), U9.74 (GND), U9.75 (GND), U9.76 (GND), U9.77 (GND), U9.78 (GND), U9.79 (GND), U9.80 (GND), U9.81 (GND), U9.82 (GND), U9.83 (GND), U9.84 (GND), U9.85 (GND), U9.86 (GND), U9.87 (GND), U9.88 (GND), U9.89 (GND), U9.91 (GND), U9.92 (GND), U9.94 (GND)
- net SIM_EAR_N: now also EAR_N.1, U9.41 (EAR_N)
- net SIM_EAR_P: now also EAR_P.1, U9.40 (EAR_P)
- net sim1_clk: now also U9.32 (USIM1_CLK); no longer U3.32 (USIM1_CLK)
- net sim1_dat: now also U9.31 (USIM1_DATA); no longer U3.31 (USIM1_DATA)
- net sim1_rst: now also U9.33 (USIM1_RST); no longer U3.33 (USIM1_RST)
- net sim1_vdd: now also U9.30 (USIM1_VDD); no longer U3.30 (USIM1_VDD)
- net at TP1.1: now also U9.22 (UART_LOG_RX); no longer U3.22 (UART_LOG_RX)
- net at C7.1, R18.2, R19.1: now also VBAT_ADC.2 (B); no longer U3.51 (VBAT_ADC)
- net at TP3.1: now also U9.27 (USB_DP); no longer U3.27 (USB_DP)
- net at TP2.1: now also U9.23 (UART_LOG_TX); no longer U3.23 (UART_LOG_TX)
- net at TP5.1: now also U9.24 (VBUS); no longer U3.24 (VBUS)
- net at D3.2 (A2), Q2.3 (C): now also PWRKEY.2 (B); no longer U3.1 (~{PWRKEY})
- net at TP4.1: now also U9.28 (USB_DM); no longer U3.28 (USB_DM)
- new net: C42.1, J2.2 (RST), R36.2, U10.3 (K_2)
- new net: C41.1, J2.3 (CLK), R35.2, U10.4 (K_3)
- new net: C40.1, J2.7 (I/O), R34.2, U10.5 (K_4)
- new net: 1V8_SIM.1 (A), U9.15 (VDD_1V8)
- new net: U9.51 (VBAT_ADC), VBAT_ADC.1 (A)
- new net: U9.55 (VBAT), U9.56 (VBAT), U9.57 (VBAT), VBAT_SIM.1 (A), VBAT_SIM1.1 (A), VBAT_SIM2.1 (A)
- new net: PWRKEY.1 (A), U9.1 (PWRKEY)
- new net: MIC_P.1, U9.42 (MIC_P)
- new net: MIC_N.1, U9.43 (MIC_N)
- new net: U9.6 (USB_BOOT), USB_BOOT.1 (A)
- new net: R33.1, USB_BOOT.2 (B)
- new net +3.3V: C46.1, U11.16 (VCCB)
- new net RI_SIM_1V8: U11.5 (1A2), U9.4 (RI)
- new net RI_SIM_3V3: U11.12 (1B2)
- new net RX_SIM_1V8: U11.6 (2A1), U9.10 (RXD)
- new net RX_SIM_3V3: U11.11 (2B1)
- new net TX_SIM_1V8: U11.4 (1A1), U9.9 (TXD)
- new net TX_SIM_3V3: U11.13 (1B1)
- new net sim2_clk: R35.1, U9.109 (USIM2_CLK)
- new net sim2_dat: R34.1, U9.108 (USIM2_DATA)
- new net sim2_rst: R36.1, U9.111 (USIM2_RST)
- new net sim2_vdd: C43.1, C44.1, J2.1 (VCC), U10.1 (K_1), U9.110 (USIM2_VDD)
- no-connect marks 54 -> 87
Other:
- moved on the sheet: C14, C15, C16, C17, C18, C7, D3, J4, Q2, R13, R14, R18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

Commit message: PCB BEGINNNING
Parts:
- removed U3: A7672SA__LASE_, symbold:XCVR_A7672SA__LASE_, symbol A7672SA__LASE_:A7672SA__LASE_
- C14, C15, C16, C17, C18, C40, C41, C42, C43, C44, C45, C46, C7: footprint (none) -> Capacitor_SMD:C_0603_1608Metric_Pad1.08x0.95mm_HandSolder
- D3: footprint (none) -> Diode_SMD:D_0603_1608Metric_Pad1.05x0.95mm_HandSolder
- EAR_N1: renamed from EAR_N; footprint (none) -> TestPoint:TestPoint_Pad_D1.5mm
- EAR_P1: renamed from EAR_P; footprint (none) -> TestPoint:TestPoint_Pad_D1.5mm
- J2, J4: footprint (none) -> Connector_Card:nanoSIM_GCT_SIM8060-6-0-14-00
- MIC_N1: renamed from MIC_N; footprint (none) -> TestPoint:TestPoint_Pad_D1.5mm
- MIC_P1: renamed from MIC_P; footprint (none) -> TestPoint:TestPoint_Pad_D1.5mm
- R13, R14, R18, R19, R20, R21, R22, R33, R34, R35, R36: footprint (none) -> Resistor_SMD:R_0603_1608Metric_Pad0.98x0.95mm_HandSolder
- TP1, TP2, TP3, TP4, TP5: footprint (none) -> TestPoint:TestPoint_Pad_D1.0mm
- U10, U5: footprint SMF15CT1G:SOT65P210X110-6N -> SMF05CT1G:SOT65P210X110-6N
- U11: footprint TSSOP16_PW_TEX -> footprints:TSSOP16_PW_TEX
- U9: footprint (none) -> a7672a:XCVR_A7672SA__LASE_
- renumbered 1V8_SIM to 1V8_SIM1, PWRKEY to PWRKEY1, USB_BOOT to USB_BOOT1, VBAT_ADC to VBAT_ADC1, VBAT_SIM to VBAT_SIM3
Connections:
- no-connect marks 87 -> 35
