File: AUDIO.kicad_sch (KiCad schematic)
At the start: 16 parts, among them J5 SJ-3524-SMT, U8 TLV320AIC3100

Commit message: mblya
Parts:
- renumbered C24 to C10, C22 to C11, C26 to C12, C27 to C13, C28 to C19, C30 to C20, C31 to C21, C19 to C22, C20 to C23, C29 to C24, C21 to C6, C25 to C8, C23 to C9, J5 to J6, U8 to U7
Other:
- moved on the sheet: J6

Commit message: SCHEMATIC
Other:
- moved on the sheet: C9
Changed lines of the file:
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@@
-	)
-	(junction
-		(at 142.24 63.5)
-		(diameter 0)
-		(color 0 0 0 0)
 	)
 	(junction
@@
 	)
 	(junction
+		(at 142.24 67.31)
+		(diameter 0)
+		(color 0 0 0 0)
+	)
+	(junction
 		(at 146.05 88.9)
 		(diameter 0)
@@
 	(wire
 		(pts
-			(xy 134.62 63.5) (xy 134.62 69.85)
+			(xy 134.62 67.31) (xy 134.62 69.85)
 		)
 		(stroke
@@
 	(wire
 		(pts
-			(xy 142.24 50.8) (xy 142.24 63.5)
-		)
-		(stroke
-			(width 0)
-			(type default)
-		)
-	)
-	(wire
-		(pts
 			(xy 146.05 130.81) (xy 146.05 134.62)
 		)
@@
 	(wire
 		(pts
-			(xy 142.24 63.5) (xy 142.24 74.93)
-		)
-		(stroke
-			(width 0)
-			(type default)
-		)
-	)
-	(wire
-		(pts
 			(xy 177.8 123.19) (xy 180.34 123.19)
 		)
@@
 	(wire
 		(pts
+			(xy 142.24 50.8) (xy 142.24 67.31)
+		)
+		(stroke
+			(width 0)
+			(type default)
+		)
+	)
+	(wire
+		(pts
 			(xy 177.8 118.11) (xy 180.34 118.11)
 		)
@@
 		(pts
 			(xy 152.4 76.2) (xy 152.4 90.17)
+		)
+		(stroke
+			(width 0)
+			(type default)
+		)
+	)
+	(wire
+		(pts
+			(xy 142.24 67.31) (xy 142.24 74.93)
 		)
 		(stroke
@@
 	(symbol
 		(lib_id "Device:C")
-		(at 138.43 63.5 90)
+		(at 138.43 67.31 90)
 		(unit 1)
 		(exclude_from_sim no)
@@
 		(dnp no)
 		(property "Reference" "C9"
-			(at 135.382 64.77 90)
+			(at 135.382 66.294 90)
 			(effects
 				(font
@@
 		)
 		(property "Value" "10uF"
-			(at 135.636 60.706 90)
+			(at 135.636 64.516 90)
 			(effects
 				(font
@@
 		)
 		(property "Footprint" ""
-			(at 142.24 62.5348 0)
+			(at 142.24 66.3448 0)
 			(effects
 				(font
@@
 		)
 		(property "Datasheet" "~"
-			(at 138.43 63.5 0)
+			(at 138.43 67.31 0)
 			(effects
 				(font
@@
 		)
 		(property "Description" "Unpolarized capacitor"
-			(at 138.43 63.5 0)
+			(at 138.43 67.31 0)
 			(effects
 				(font
@@
 		(dnp no)
 		(property "Reference" "C10"
-			(at 134.366 76.708 90)
+			(at 134.874 76.454 90)
 			(effects
 				(font
@@
 		)
 		(property "Value" "100nF"
-			(at 133.858 73.406 90)
-			(effects
-				(font
+			(at 135.89 78.74 90)
+			(effects
+				(font

Commit message: PCB BEGINNNING
Parts:
- C10, C11, C12, C13, C19, C20, C21, C22, C23, C24, C6, C8, C9: footprint (none) -> Capacitor_SMD:C_0603_1608Metric_Pad1.08x0.95mm_HandSolder
- J6: footprint SJ-3524-SMT:CUI_SJ-3524-SMT -> Connector_Audio:Jack_3.5mm_CUI_SJ-3524-SMT_Horizontal
- LS1: footprint (none) -> Connector_JST:JST_EH_B2B-EH-A_1x02_P2.50mm_Vertical
Connections:
- net +VSW renamed +BATT
Changed lines of the file:
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@@
 			)
 		)
-		(property "Footprint" ""
+		(property "Footprint" "Connector_JST:JST_EH_B2B-EH-A_1x02_P2.50mm_Vertical"
 			(at 184.15 101.6 0)
 			(effects
@@
 			)
 		)
-		(property "Footprint" ""
+		(property "Footprint" "Capacitor_SMD:C_0603_1608Metric_Pad1.08x0.95mm_HandSolder"
 			(at 175.26 106.9848 0)
 			(effects
@@
 			)
 		)
-		(property "Footprint" "SJ-3524-SMT:CUI_SJ-3524-SMT"
+		(property "Footprint" "Connector_Audio:Jack_3.5mm_CUI_SJ-3524-SMT_Horizontal"
 			(at 227.33 104.14 0)
 			(effects
@@
 			)
 		)
-		(property "Value" "+VSW"
+		(property "Value" "+BATT"
 			(at 180.34 66.04 0)
 			(effects
@@
 			)
 		)
-		(property "Footprint" ""
+		(property "Footprint" "Capacitor_SMD:C_0603_1608Metric_Pad1.08x0.95mm_HandSolder"
 			(at 159.0548 76.2 0)
 			(effects
@@
 			)
 		)
-		(property "Footprint" ""
+		(property "Footprint" "Capacitor_SMD:C_0603_1608Metric_Pad1.08x0.95mm_HandSolder"
 			(at 142.24 66.3448 0)
 			(effects
@@
 			)
 		)
-		(property "Footprint" ""
+		(property "Footprint" "Capacitor_SMD:C_0603_1608Metric_Pad1.08x0.95mm_HandSolder"
 			(at 177.8 122.2248 0)
 			(effects
@@
 			)
 		)
-		(property "Footprint" ""
+		(property "Footprint" "Capacitor_SMD:C_0603_1608Metric_Pad1.08x0.95mm_HandSolder"
 			(at 154.94 70.1548 0)
 			(effects
@@
 			)
 		)
-		(property "Footprint" ""
+		(property "Footprint" "Capacitor_SMD:C_0603_1608Metric_Pad1.08x0.95mm_HandSolder"
 			(at 170.4848 76.2 0)
 			(effects
@@
 			)
 		)
-		(property "Footprint" ""
+		(property "Footprint" "Capacitor_SMD:C_0603_1608Metric_Pad1.08x0.95mm_HandSolder"
 			(at 176.8348 76.2 0)
 			(effects
@@
 			)
 		)
-		(property "Footprint" ""
+		(property "Footprint" "Capacitor_SMD:C_0603_1608Metric_Pad1.08x0.95mm_HandSolder"
 			(at 175.26 109.5248 0)
 			(effects
@@
 			)
 		)
-		(property "Footprint" ""
+		(property "Footprint" "Capacitor_SMD:C_0603_1608Metric_Pad1.08x0.95mm_HandSolder"
 			(at 124.46 79.0448 0)
 			(effects
@@
 			)
 		)
-		(property "Footprint" ""
+		(property "Footprint" "Capacitor_SMD:C_0603_1608Metric_Pad1.08x0.95mm_HandSolder"
 			(at 177.8 117.1448 0)
 			(effects
@@
 			)
 		)
-		(property "Footprint" ""
+		(property "Footprint" "Capacitor_SMD:C_0603_1608Metric_Pad1.08x0.95mm_HandSolder"
 			(at 164.1348 76.2 0)
 			(effects
@@
 			)
 		)
-		(property "Footprint" ""
+		(property "Footprint" "Capacitor_SMD:C_0603_1608Metric_Pad1.08x0.95mm_HandSolder"
 			(at 142.24 73.9648 0)
 			(effects
@@
 			)
 		)
-		(property "Footprint" ""
+		(property "Footprint" "Capacitor_SMD:C_0603_1608Metric_Pad1.08x0.95mm_HandSolder"
 			(at 124.46 84.1248 0)
 			(effects

Commit message: lol
Connections:
- net GND: now also J6.1; no longer J6.2
- net at C20.2: now also J6.2; no longer J6.1
- net at J6.4: no longer U7.11 (VOL/MICDET)
- no-connect marks 2 -> 4
Changed lines of the file:
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@@
 		(at 167.64 120.65)
 	)
+	(no_connect
+		(at 167.64 115.57)
+	)
+	(no_connect
+		(at 204.47 104.14)
+	)
 	(wire
 		(pts
@@
 	(wire
 		(pts
+			(xy 175.26 101.6) (xy 214.63 101.6)
+		)
+		(stroke
+			(width 0)
+			(type default)
+		)
+	)
+	(wire
+		(pts
 			(xy 146.05 130.81) (xy 146.05 134.62)
 		)
@@
 	(wire
 		(pts
-			(xy 175.26 107.95) (xy 214.63 107.95)
-		)
-		(stroke
-			(width 0)
-			(type default)
-		)
-	)
-	(wire
-		(pts
 			(xy 149.86 90.17) (xy 152.4 90.17)
 		)
@@
 	(wire
 		(pts
-			(xy 205.74 101.6) (xy 214.63 101.6)
-		)
-		(stroke
-			(width 0)
-			(type default)
-		)
-	)
-	(wire
-		(pts
 			(xy 116.84 80.01) (xy 113.03 80.01)
 		)
@@
 	(wire
 		(pts
+			(xy 175.26 101.6) (xy 175.26 107.95)
+		)
+		(stroke
+			(width 0)
+			(type default)
+		)
+	)
+	(wire
+		(pts
 			(xy 182.88 87.63) (xy 182.88 88.9)
 		)
@@
 	(wire
 		(pts
-			(xy 204.47 104.14) (xy 204.47 115.57)
-		)
-		(stroke
-			(width 0)
-			(type default)
-		)
-	)
-	(wire
-		(pts
 			(xy 124.46 85.09) (xy 124.46 88.9)
 		)
@@
 	(wire
 		(pts
+			(xy 201.93 107.95) (xy 214.63 107.95)
+		)
+		(stroke
+			(width 0)
+			(type default)
+		)
+	)
+	(wire
+		(pts
 			(xy 204.47 104.14) (xy 214.63 104.14)
 		)
@@
 		(pts
 			(xy 167.64 118.11) (xy 170.18 118.11)
-		)
-		(stroke
-			(width 0)
-			(type default)
-		)
-	)
-	(wire
-		(pts
-			(xy 204.47 115.57) (xy 167.64 115.57)
 		)
 		(stroke
@@
 	(symbol
 		(lib_id "power:GND")
-		(at 205.74 101.6 270)
+		(at 201.93 107.95 270)
 		(unit 1)
 		(exclude_from_sim no)
@@
 		(fields_autoplaced yes)
 		(property "Reference" "#PWR047"
-			(at 199.39 101.6 0)
+			(at 195.58 107.95 0)
 			(effects
 				(font
@@
 		)
 		(property "Value" "GND"
-			(at 201.93 101.5999 90)
+			(at 198.12 107.9499 90)
 			(effects
 				(font
@@
 		)
 		(property "Footprint" ""
-			(at 205.74 101.6 0)
+			(at 201.93 107.95 0)
 			(effects
 				(font
@@
 		)
 		(property "Datasheet" ""
-			(at 205.74 101.6 0)
+			(at 201.93 107.95 0)
 			(effects
 				(font
@@
 		)
 		(property "Description" "Power symbol creates a global label with name \"GND\" , ground"
-			(at 205.74 101.6 0)
-			(effects
-				(font
+			(at 201.93 107.95 0)
+			(effects
+				(font

Commit message: P
Parts:
- added C49: 100nF, Capacitor_SMD:C_0603_1608Metric_Pad1.08x0.95mm_HandSolder, symbol Device:C
- added JP1, JP2: SolderJumper_2_Open, Jumper:SolderJumper-2_P1.3mm_Open_TrianglePad1.0x1.5mm, symbol Jumper:SolderJumper_2_Open
- added R41: 2.2k, symbol Device:R
- J6: footprint Connector_Audio:Jack_3.5mm_CUI_SJ-3524-SMT_Horizontal -> 35RASMT6CHNTRX:SWITCHCRAFT_35RASMT6CHNTRX; symbol SJ-3524-SMT:SJ-3524-SMT -> 35RASMT6CHNTRX:35RASMT6CHNTRX; MANUFACTURER (none) -> Switchcraft; MAXIMUM_PACKAGE_HEIGHT (none) -> 5.1mm; PARTREV 1.03 -> A; STANDARD Manufacturer recommendations -> Manufacturer Recommendations
Connections:
- net GND: now also JP1.1 (A); no longer J6.1
- net at J6.4: now also JP2.2 (B)
- net at U7.11 (VOL/MICDET): now also C49.1, JP2.1 (A), R41.2
- net at U7.12 (MICBIAS): now also R41.1
- net at U7.14 (MIC1RP): now also C49.2
- new net: J6.1, JP1.2 (B)
- no-connect marks 4 -> 0
