File: okabephone.kicad_pcb (KiCad board)
At the start: 2 copper layers, 49 x 120 mm, 3 parts, among them U1 MCP23017_ML, U2 ESP32-S3-WROOM-1, U3 AMS1117-3.3

Commit message: spi joke
Parts:
- removed U1: MCP23017_ML, Package_DFN_QFN:QFN-28-1EP_6x6mm_P0.65mm_EP4.25x4.25mm
- removed U2: ESP32-S3-WROOM-1, RF_Module:ESP32-S3-WROOM-1
- removed U3: AMS1117-3.3, Package_TO_SOT_SMD:SOT-223-3_TabPin2

Commit message: :)
Parts:
- added C1: 4.7uF, Capacitor_SMD:C_0603_1608Metric, F.Cu at (238.7, 129.4)
- added C13: 22uF 16V X5R, Capacitor_SMD:C_1206_3216Metric, F.Cu at (255.0, 128.0)
- added C2: 0-8.2pF, Capacitor_SMD:C_0603_1608Metric_Pad1.08x0.95mm_HandSolder, F.Cu at (257.0, 121.7)
- added D2: SS14, Diode_SMD:D_SMA, F.Cu at (206.8, 119.3)
- added D4: BAV70, Package_TO_SOT_SMD:SOT-23, F.Cu at (247.7, 113.8)
- added J3: BATTERY, OKPH:Battery connector 3mm nergon, F.Cu at (224.3, 123.3)
- added J6: SFH11-PBPC-D10-RA-BK, connector:CONN20_D10-RA-BK_SUL, F.Cu at (223.0, 23.5)
- added L1: 2.2uH, Inductor_SMD:L_6.3x6.3_H3, F.Cu at (254.4, 115.5)
- added Q1: AO3400A, Package_TO_SOT_SMD:SOT-23, F.Cu at (213.3, 119.2)
- added Q2: BC847, Package_TO_SOT_SMD:SOT-23, F.Cu at (185.7, 82.0)
- added Q3: IRLML6402, Package_TO_SOT_SMD:SOT-23, F.Cu at (247.7, 118.2)
- added R4: 5.1k, Capacitor_SMD:C_0603_1608Metric_Pad1.08x0.95mm_HandSolder, F.Cu at (257.0, 124.2)
- added TH1: NTC, Connector_JST:JST_EH_B2B-EH-A_1x02_P2.50mm_Vertical, F.Cu at (268.5, 123.5)
- added U1: MCP23017_ML, Package_DFN_QFN:QFN-28-1EP_6x6mm_P0.65mm_EP4.25x4.25mm, F.Cu at (190.2, 121.1)
- added U2: ESP32-S3-WROOM-1, RF_Module:ESP32-S3-WROOM-1U, F.Cu at (197.1, 39.5)
- added U3: A7672SA__LASE_, symbold:XCVR_A7672SA__LASE_, F.Cu at (201.7, 68.6)
- added U4: BQ21040DBV, Package_TO_SOT_SMD:SOT-23-6, F.Cu at (239.3, 125.9)
- added U6: PCF8563T, Package_SO:SOIC-8_3.9x4.9mm_P1.27mm, F.Cu at (198.5, 120.3)
- added U7: RT8059, Package_TO_SOT_SMD:TSOT-23-5_HandSoldering, F.Cu at (248.7, 128.7)
- added U8: TLV320AIC3100, Package_DFN_QFN:VQFN-32-1EP_5x5mm_P0.5mm_EP3.5x3.5mm, F.Cu at (189.7, 130.9)
- added Y1: 32.768kHz, Crystal:Crystal_SMD_3215-2Pin_3.2x1.5mm, F.Cu at (205.3, 123.2)
Other:
- board text added: "NOKIA BATTERY"

Commit message: PCB BEGINNNING
Parts:
- removed U3: A7672SA__LASE_, symbold:XCVR_A7672SA__LASE_
- removed Y1: 32.768kHz, Crystal:Crystal_SMD_3215-2Pin_3.2x1.5mm
- added 1V8_SIM1: SolderJumper_2_Open, Jumper:SolderJumper-2_P1.3mm_Open_Pad1.0x1.5mm, F.Cu at (255.5, 75.3)
- added BUCK_BAT1: SolderJumper_2_Open, Jumper:SolderJumper-2_P1.3mm_Open_Pad1.0x1.5mm, F.Cu at (266.8, 75.3)
- added BUCK_POST1: SolderJumper_2_Open, Jumper:SolderJumper-2_P1.3mm_Open_Pad1.0x1.5mm, F.Cu at (266.8, 78.9)
- added BUCK_VBUS1: SolderJumper_2_Open, Jumper:SolderJumper-2_P1.3mm_Open_Pad1.0x1.5mm, F.Cu at (266.8, 82.5)
- added C10: 100nF, Capacitor_SMD:C_0603_1608Metric_Pad1.08x0.95mm_HandSolder, F.Cu at (354.0, 158.7)
- added C11: 22uF, Capacitor_SMD:C_0603_1608Metric_Pad1.08x0.95mm_HandSolder, F.Cu at (354.0, 161.2)
- added C12: 22uF, Capacitor_SMD:C_0603_1608Metric_Pad1.08x0.95mm_HandSolder, F.Cu at (358.3, 151.1)
- added C14: 22pF, Capacitor_SMD:C_0603_1608Metric_Pad1.08x0.95mm_HandSolder, F.Cu at (306.6, 170.1)
- added C15: 22pF, Capacitor_SMD:C_0603_1608Metric_Pad1.08x0.95mm_HandSolder, F.Cu at (306.6, 172.6)
- added C16: 22pF, Capacitor_SMD:C_0603_1608Metric_Pad1.08x0.95mm_HandSolder, F.Cu at (306.6, 175.1)
- added C17: 100nF, Capacitor_SMD:C_0603_1608Metric_Pad1.08x0.95mm_HandSolder, F.Cu at (306.6, 177.6)
- added C18: 33pF, Capacitor_SMD:C_0603_1608Metric_Pad1.08x0.95mm_HandSolder, F.Cu at (306.6, 180.1)
- added C19: 100nF, Capacitor_SMD:C_0603_1608Metric_Pad1.08x0.95mm_HandSolder, F.Cu at (358.3, 156.2)
- added C20: 47uF, Capacitor_SMD:C_0603_1608Metric_Pad1.08x0.95mm_HandSolder, F.Cu at (358.3, 158.7)
- added C21: 47uF, Capacitor_SMD:C_0603_1608Metric_Pad1.08x0.95mm_HandSolder, F.Cu at (358.3, 161.2)
- added C22: 1uF, Capacitor_SMD:C_0603_1608Metric_Pad1.08x0.95mm_HandSolder, F.Cu at (362.7, 151.1)
- added C23: 1uF, Capacitor_SMD:C_0603_1608Metric_Pad1.08x0.95mm_HandSolder, F.Cu at (362.7, 153.6)
- added C24: 100nF, Capacitor_SMD:C_0603_1608Metric_Pad1.08x0.95mm_HandSolder, F.Cu at (362.7, 156.2)
- added C25: 10uF, Capacitor_SMD:C_0603_1608Metric_Pad1.08x0.95mm_HandSolder, F.Cu at (344.1, 116.8)
- added C26: 100nF, Capacitor_SMD:C_0603_1608Metric_Pad1.08x0.95mm_HandSolder, F.Cu at (344.1, 119.4)
- added C27: 10uF, Capacitor_SMD:C_0603_1608Metric_Pad1.08x0.95mm_HandSolder, F.Cu at (344.1, 121.9)
- added C28: 100nF, Capacitor_SMD:C_0603_1608Metric_Pad1.08x0.95mm_HandSolder, F.Cu at (344.1, 124.4)
- added C29: 10uF, Capacitor_SMD:C_0603_1608Metric_Pad1.08x0.95mm_HandSolder, F.Cu at (344.1, 126.9)
- added C3: 4.7uF, Capacitor_SMD:C_0603_1608Metric_Pad1.08x0.95mm_HandSolder, F.Cu at (266.6, 89.0)
- added C30: 100nF, Capacitor_SMD:C_0603_1608Metric_Pad1.08x0.95mm_HandSolder, F.Cu at (344.1, 129.4)
- added C31: 10uF, Capacitor_SMD:C_0603_1608Metric_Pad1.08x0.95mm_HandSolder, F.Cu at (344.1, 131.9)
- added C32: 100nF, Capacitor_SMD:C_0603_1608Metric_Pad1.08x0.95mm_HandSolder, F.Cu at (344.1, 134.4)
- added C33: 10uF, Capacitor_SMD:C_0603_1608Metric_Pad1.08x0.95mm_HandSolder, F.Cu at (348.4, 116.8)
- added C34: 100nF, Capacitor_SMD:C_0603_1608Metric_Pad1.08x0.95mm_HandSolder, F.Cu at (348.4, 119.4)
- added C35: 100nF, Capacitor_SMD:C_0603_1608Metric_Pad1.08x0.95mm_HandSolder, F.Cu at (348.4, 121.9)
- added C36: 100nF, Capacitor_SMD:C_0603_1608Metric_Pad1.08x0.95mm_HandSolder, F.Cu at (348.4, 124.4)
- added C37: 1uF, Capacitor_SMD:C_0603_1608Metric_Pad1.08x0.95mm_HandSolder, F.Cu at (348.4, 126.9)
- added C38: NC, Capacitor_SMD:C_0603_1608Metric_Pad1.08x0.95mm_HandSolder, F.Cu at (348.4, 129.4)
- added C39: NC, Capacitor_SMD:C_0603_1608Metric_Pad1.08x0.95mm_HandSolder, F.Cu at (348.4, 131.9)
- added C4: 0-8.2pF, Capacitor_SMD:C_0603_1608Metric_Pad1.08x0.95mm_HandSolder, F.Cu at (271.1, 92.6)
- added C40: 22pF, Capacitor_SMD:C_0603_1608Metric_Pad1.08x0.95mm_HandSolder, F.Cu at (310.9, 167.6)
- added C41: 22pF, Capacitor_SMD:C_0603_1608Metric_Pad1.08x0.95mm_HandSolder, F.Cu at (310.9, 170.1)
- added C42: 22pF, Capacitor_SMD:C_0603_1608Metric_Pad1.08x0.95mm_HandSolder, F.Cu at (310.9, 172.6)
- added C43: 100nF, Capacitor_SMD:C_0603_1608Metric_Pad1.08x0.95mm_HandSolder, F.Cu at (310.9, 175.1)
- added C44: 33pF, Capacitor_SMD:C_0603_1608Metric_Pad1.08x0.95mm_HandSolder, F.Cu at (310.9, 177.6)
- added C45: 100nF, Capacitor_SMD:C_0603_1608Metric_Pad1.08x0.95mm_HandSolder, F.Cu at (310.9, 180.1)
- added C46: 100nF, Capacitor_SMD:C_0603_1608Metric_Pad1.08x0.95mm_HandSolder, F.Cu at (315.3, 167.6)
- added C5: 22uF 16V X5R, Capacitor_SMD:C_1206_3216Metric, F.Cu at (280.3, 83.1)
- added C6: 10uF, Capacitor_SMD:C_0603_1608Metric_Pad1.08x0.95mm_HandSolder, F.Cu at (354.0, 151.1)
- added C7: 1uF, Capacitor_SMD:C_0603_1608Metric_Pad1.08x0.95mm_HandSolder, F.Cu at (306.6, 167.6)
- added C8: 100nF, Capacitor_SMD:C_0603_1608Metric_Pad1.08x0.95mm_HandSolder, F.Cu at (354.0, 153.6)
- added C9: 10uF, Capacitor_SMD:C_0603_1608Metric_Pad1.08x0.95mm_HandSolder, F.Cu at (354.0, 156.2)
- added CHRG_VBUS1: SolderJumper_2_Open, Jumper:SolderJumper-2_P1.3mm_Open_Pad1.0x1.5mm, F.Cu at (266.8, 86.0)
- added D1: BAV70, Package_TO_SOT_SMD:SOT-23, F.Cu at (275.8, 93.7)
- added D10: D_TVS, Diode_SMD:D_0603_1608Metric_Pad1.05x0.95mm_HandSolder, F.Cu at (347.2, 144.7)
- added D3: D_TVS, Diode_SMD:D_0603_1608Metric_Pad1.05x0.95mm_HandSolder, F.Cu at (335.1, 174.4)
- added D5: D_TVS, Diode_SMD:D_0603_1608Metric_Pad1.05x0.95mm_HandSolder, F.Cu at (382.7, 98.5)
- added D6: 1N5819WS, Diode_SMD:D_SOD-323, F.Cu at (271.7, 114.1)
- added D7: D_TVS, Diode_SMD:D_0603_1608Metric_Pad1.05x0.95mm_HandSolder, F.Cu at (347.2, 137.0)
- added D8: D_TVS, Diode_SMD:D_0603_1608Metric_Pad1.05x0.95mm_HandSolder, F.Cu at (347.2, 139.6)
- added D9: D_TVS, Diode_SMD:D_0603_1608Metric_Pad1.05x0.95mm_HandSolder, F.Cu at (347.2, 142.2)
- added EAR_N1: TestPoint, TestPoint:TestPoint_Pad_D1.5mm, F.Cu at (326.6, 168.1)
- added EAR_P1: TestPoint, TestPoint:TestPoint_Pad_D1.5mm, F.Cu at (326.6, 171.7)
- added F1: Polyfuse, Fuse:Fuse_1210_3225Metric, F.Cu at (377.2, 110.1)
- added J1: Micro_SD_Card_Det1, Connector_Card:microSD_HC_Hirose_DM3AT-SF-PEJM5, F.Cu at (350.3, 101.3)
- added J2: SIM_Card, Connector_Card:nanoSIM_GCT_SIM8060-6-0-14-00, F.Cu at (312.2, 158.3)
- added J4: SIM_Card, Connector_Card:nanoSIM_GCT_SIM8060-6-0-14-00, F.Cu at (327.9, 158.3)
- added J5: USB_C_Receptacle_USB2.0_16P, UJ20-C-G-MSMT-TR-68:CUI_UJ20-C-G-MSMT-TR-68, F.Cu at (210.2, 134.6)
- added J7: Conn_01x12_MountingPin, Connector_FFC-FPC:TE_1-1734839-2_1x12-1MP_P0.5mm_Horizontal, F.Cu at (208.8, 45.9)
- added LS1: Speaker, Connector_JST:JST_EH_B2B-EH-A_1x02_P2.50mm_Vertical, F.Cu at (212.8, 20.7)
- added M1: Motor_DC, Connector_JST:JST_EH_B2B-EH-A_1x02_P2.50mm_Vertical, F.Cu at (352.9, 138.3)
- added MIC_N1: TestPoint, TestPoint:TestPoint_Pad_D1.5mm, F.Cu at (326.6, 175.2)
- added MIC_P1: TestPoint, TestPoint:TestPoint_Pad_D1.5mm, F.Cu at (326.6, 178.8)
- added PWRKEY1: SolderJumper_2_Open, Jumper:SolderJumper-2_P1.3mm_Open_Pad1.0x1.5mm, F.Cu at (255.5, 78.9)
- added R1: 10k, Resistor_SMD:R_0603_1608Metric_Pad0.98x0.95mm_HandSolder, F.Cu at (348.4, 134.4)
- added R10: 10k, Resistor_SMD:R_0603_1608Metric_Pad0.98x0.95mm_HandSolder, F.Cu at (372.2, 105.4)
- added R11: 249k, Resistor_SMD:R_0603_1608Metric_Pad0.98x0.95mm_HandSolder, F.Cu at (372.2, 107.9)
- added R12: 54.9k, Resistor_SMD:R_0603_1608Metric_Pad0.98x0.95mm_HandSolder, F.Cu at (372.2, 110.4)
- added R13: 4.7k, Resistor_SMD:R_0603_1608Metric_Pad0.98x0.95mm_HandSolder, F.Cu at (315.3, 170.1)
- added R14: 4.7k, Resistor_SMD:R_0603_1608Metric_Pad0.98x0.95mm_HandSolder, F.Cu at (315.3, 172.6)
- added R15: 22, Resistor_SMD:R_0603_1608Metric_Pad0.98x0.95mm_HandSolder, F.Cu at (352.8, 116.8)
- added R16: 22, Resistor_SMD:R_0603_1608Metric_Pad0.98x0.95mm_HandSolder, F.Cu at (352.8, 119.4)
- added R17: 10k, Resistor_SMD:R_0603_1608Metric_Pad0.98x0.95mm_HandSolder, F.Cu at (352.8, 121.9)
- added R18: 680k, Resistor_SMD:R_0603_1608Metric_Pad0.98x0.95mm_HandSolder, F.Cu at (315.3, 175.1)
- added R19: 470k, Resistor_SMD:R_0603_1608Metric_Pad0.98x0.95mm_HandSolder, F.Cu at (315.3, 177.6)
- added R2: 680, Resistor_SMD:R_0603_1608Metric_Pad0.98x0.95mm_HandSolder, F.Cu at (363.5, 107.9)
- added R20: 22, Resistor_SMD:R_0603_1608Metric_Pad0.98x0.95mm_HandSolder, F.Cu at (315.3, 180.1)
- added R21: 22, Resistor_SMD:R_0603_1608Metric_Pad0.98x0.95mm_HandSolder, F.Cu at (319.6, 167.6)
- added R22: 22, Resistor_SMD:R_0603_1608Metric_Pad0.98x0.95mm_HandSolder, F.Cu at (319.6, 170.1)
- added R23: 10k, Resistor_SMD:R_0603_1608Metric_Pad0.98x0.95mm_HandSolder, F.Cu at (352.8, 124.4)
- added R24: 1k, Resistor_SMD:R_0603_1608Metric_Pad0.98x0.95mm_HandSolder, F.Cu at (352.8, 126.9)
- added R25: 200k, Resistor_SMD:R_0603_1608Metric_Pad0.98x0.95mm_HandSolder, F.Cu at (352.8, 129.4)
- added R26: 6.8, Resistor_SMD:R_0603_1608Metric_Pad0.98x0.95mm_HandSolder, F.Cu at (352.8, 131.9)
- added R27: NC, Resistor_SMD:R_0603_1608Metric_Pad0.98x0.95mm_HandSolder, F.Cu at (352.8, 134.4)
- added R28: 10k, Resistor_SMD:R_0603_1608Metric_Pad0.98x0.95mm_HandSolder, F.Cu at (357.1, 116.8)
- added R29: 10k, Resistor_SMD:R_0603_1608Metric_Pad0.98x0.95mm_HandSolder, F.Cu at (357.1, 119.4)
- added R3: 10k, Resistor_SMD:R_0603_1608Metric_Pad0.98x0.95mm_HandSolder, F.Cu at (363.5, 110.4)
- added R30: 10k, Resistor_SMD:R_0603_1608Metric_Pad0.98x0.95mm_HandSolder, F.Cu at (357.1, 121.9)
- added R31: 10k, Resistor_SMD:R_0603_1608Metric_Pad0.98x0.95mm_HandSolder, F.Cu at (357.1, 124.4)
- added R32: 10k, Resistor_SMD:R_0603_1608Metric_Pad0.98x0.95mm_HandSolder, F.Cu at (357.1, 126.9)
- added R33: 10k, Resistor_SMD:R_0603_1608Metric_Pad0.98x0.95mm_HandSolder, F.Cu at (319.6, 172.6)
- added R34: 22, Resistor_SMD:R_0603_1608Metric_Pad0.98x0.95mm_HandSolder, F.Cu at (319.6, 175.1)
- added R35: 22, Resistor_SMD:R_0603_1608Metric_Pad0.98x0.95mm_HandSolder, F.Cu at (319.6, 177.6)
- added R36: 22, Resistor_SMD:R_0603_1608Metric_Pad0.98x0.95mm_HandSolder, F.Cu at (319.6, 180.1)
- added R37: 10k, Resistor_SMD:R_0603_1608Metric_Pad0.98x0.95mm_HandSolder, F.Cu at (357.1, 129.4)
- added R38: 470, Resistor_SMD:R_0603_1608Metric_Pad0.98x0.95mm_HandSolder, F.Cu at (357.1, 131.9)
- added R5: 100k, Resistor_SMD:R_0603_1608Metric_Pad0.98x0.95mm_HandSolder, F.Cu at (367.8, 105.4)
- added R6: 5.1k, Resistor_SMD:R_0603_1608Metric_Pad0.98x0.95mm_HandSolder, F.Cu at (271.1, 95.1)
- added R7: 5.1k, Resistor_SMD:R_0603_1608Metric_Pad0.98x0.95mm_HandSolder, F.Cu at (367.8, 107.9)
- added R8: 100k, Resistor_SMD:R_0603_1608Metric_Pad0.98x0.95mm_HandSolder, F.Cu at (367.8, 110.4)
- added R9: 1k, Resistor_SMD:R_0603_1608Metric_Pad0.98x0.95mm_HandSolder, F.Cu at (372.2, 102.9)
- added RXD1: TestPoint, TestPoint:TestPoint_Pad_D1.0mm, F.Cu at (343.4, 137.2)
- added SW1: SW_MEC_5E, PTS526_SM08_SMTR2_LFS:SW_PTS526_SM08_SMTR2_LFS, F.Cu at (309.5, 95.2)
- added SW10: SW_MEC_5E, PTS526_SM08_SMTR2_LFS:SW_PTS526_SM08_SMTR2_LFS, F.Cu at (318.9, 107.8)
- added SW11: SW_MEC_5E, PTS526_SM08_SMTR2_LFS:SW_PTS526_SM08_SMTR2_LFS, F.Cu at (318.9, 114.2)
- added SW12: SW_MEC_5E, PTS526_SM08_SMTR2_LFS:SW_PTS526_SM08_SMTR2_LFS, F.Cu at (318.9, 120.5)
- added SW13: SW_MEC_5E, PTS526_SM08_SMTR2_LFS:SW_PTS526_SM08_SMTR2_LFS, F.Cu at (318.9, 126.9)
- added SW14: SW_MEC_5E, PTS526_SM08_SMTR2_LFS:SW_PTS526_SM08_SMTR2_LFS, F.Cu at (318.9, 133.2)
- added SW15: SW_MEC_5E, PTS526_SM08_SMTR2_LFS:SW_PTS526_SM08_SMTR2_LFS, F.Cu at (328.3, 95.2)
- added SW16: SW_MEC_5E, PTS526_SM08_SMTR2_LFS:SW_PTS526_SM08_SMTR2_LFS, F.Cu at (328.3, 101.5)
- added SW17: SW_MEC_5E, PTS526_SM08_SMTR2_LFS:SW_PTS526_SM08_SMTR2_LFS, F.Cu at (328.3, 107.8)
- added SW18: SW_MEC_5E, PTS526_SM08_SMTR2_LFS:SW_PTS526_SM08_SMTR2_LFS, F.Cu at (328.3, 114.2)
- added SW19: SW_MEC_5E, PTS526_SM08_SMTR2_LFS:SW_PTS526_SM08_SMTR2_LFS, F.Cu at (328.3, 120.5)
- added SW2: SW_MEC_5E, PTS526_SM08_SMTR2_LFS:SW_PTS526_SM08_SMTR2_LFS, F.Cu at (309.5, 101.5)
- added SW20: POWER_BUTTON, PTS526_SM08_SMTR2_LFS:SW_PTS526_SM08_SMTR2_LFS, F.Cu at (379.5, 104.8)
- added SW21: SW_MEC_5E, PTS526_SM08_SMTR2_LFS:SW_PTS526_SM08_SMTR2_LFS, F.Cu at (328.3, 126.9)
- added SW22: SW_MEC_5E, PTS526_SM08_SMTR2_LFS:SW_PTS526_SM08_SMTR2_LFS, F.Cu at (328.3, 133.2)
- added SW23: SW_MEC_5E, PTS526_SM08_SMTR2_LFS:SW_PTS526_SM08_SMTR2_LFS, F.Cu at (337.6, 95.2)
- added SW3: SW_MEC_5E, PTS526_SM08_SMTR2_LFS:SW_PTS526_SM08_SMTR2_LFS, F.Cu at (309.5, 107.8)
- added SW4: SW_MEC_5E, PTS526_SM08_SMTR2_LFS:SW_PTS526_SM08_SMTR2_LFS, F.Cu at (309.5, 114.2)
- added SW5: SW_MEC_5E, PTS526_SM08_SMTR2_LFS:SW_PTS526_SM08_SMTR2_LFS, F.Cu at (309.5, 120.5)
- added SW6: SW_MEC_5E, PTS526_SM08_SMTR2_LFS:SW_PTS526_SM08_SMTR2_LFS, F.Cu at (309.5, 126.9)
- added SW7: SW_MEC_5E, PTS526_SM08_SMTR2_LFS:SW_PTS526_SM08_SMTR2_LFS, F.Cu at (309.5, 133.2)
- added SW8: SW_MEC_5E, PTS526_SM08_SMTR2_LFS:SW_PTS526_SM08_SMTR2_LFS, F.Cu at (318.9, 95.2)
- added SW9: SW_MEC_5E, PTS526_SM08_SMTR2_LFS:SW_PTS526_SM08_SMTR2_LFS, F.Cu at (318.9, 101.5)
- added SW_BOOT1: SW_MEC_5E, PTS526_SM08_SMTR2_LFS:SW_PTS526_SM08_SMTR2_LFS, F.Cu at (337.6, 101.5)
- added SW_RST1: SW_MEC_5E, PTS526_SM08_SMTR2_LFS:SW_PTS526_SM08_SMTR2_LFS, F.Cu at (337.6, 107.8)
- added TP1: S_LOGR, TestPoint:TestPoint_Pad_D1.0mm, F.Cu at (323.3, 167.8)
- added TP2: S_LOGT, TestPoint:TestPoint_Pad_D1.0mm, F.Cu at (323.3, 170.9)
- added TP3: S_USBP, TestPoint:TestPoint_Pad_D1.0mm, F.Cu at (323.3, 173.9)
- added TP4: S_USBM, TestPoint:TestPoint_Pad_D1.0mm, F.Cu at (323.3, 177.0)
- added TP5: S_VBUS, TestPoint:TestPoint_Pad_D1.0mm, F.Cu at (323.3, 180.1)
- added TP7: BATTERY, TestPoint:TestPoint_Pad_D1.0mm, F.Cu at (381.5, 109.5)
- added TP8: 3.3V, TestPoint:TestPoint_Pad_D1.0mm, F.Cu at (343.4, 140.2)
- added TP9: GND, TestPoint:TestPoint_Pad_D1.0mm, F.Cu at (343.4, 143.3)
- added TXD1: TestPoint, TestPoint:TestPoint_Pad_D1.0mm, F.Cu at (343.4, 146.3)
- added U10: SMF15CT1G, SMF05CT1G:SOT65P210X110-6N, F.Cu at (330.7, 178.7)
- added U11: SN74AXC4T245PWR, footprints:TSSOP16_PW_TEX, F.Cu at (193.0, 68.0)
- added U5: SMF15CT1G, SMF05CT1G:SOT65P210X110-6N, F.Cu at (330.7, 175.0)
- added U9: ~, a7672a:XCVR_A7672SA__LASE_, F.Cu at (212.5, 68.0)
- added USB_BOOT1: SolderJumper_2_Open, Jumper:SolderJumper-2_P1.3mm_Open_Pad1.0x1.5mm, F.Cu at (255.5, 82.5)
- added VBAT_ADC1: SolderJumper_2_Open, Jumper:SolderJumper-2_P1.3mm_Open_Pad1.0x1.5mm, F.Cu at (255.5, 86.0)
- added VBAT_SIM1: SolderJumper_2_Open, Jumper:SolderJumper-2_P1.3mm_Open_Pad1.0x1.5mm, F.Cu at (255.5, 89.5)
- added VBAT_SIM2: SolderJumper_2_Open, Jumper:SolderJumper-2_P1.3mm_Open_Pad1.0x1.5mm, F.Cu at (255.5, 93.1)
- added VBAT_SIM3: SolderJumper_2_Open, Jumper:SolderJumper-2_P1.3mm_Open_Pad1.0x1.5mm, F.Cu at (255.5, 96.7)
- C1: value 4.7uF -> 1uF; footprint Capacitor_SMD:C_0603_1608Metric -> Capacitor_SMD:C_0603_1608Metric_Pad1.08x0.95mm_HandSolder
- C13: value 22uF 16V X5R -> 22uF; footprint Capacitor_SMD:C_1206_3216Metric -> Capacitor_SMD:C_0603_1608Metric_Pad1.08x0.95mm_HandSolder
- C2: value 0-8.2pF -> 1uF
- D2: value SS14 -> D_TVS; footprint Diode_SMD:D_SMA -> Diode_SMD:D_0603_1608Metric_Pad1.05x0.95mm_HandSolder
- D4: value BAV70 -> D_TVS; footprint Package_TO_SOT_SMD:SOT-23 -> Diode_SMD:D_0603_1608Metric_Pad1.05x0.95mm_HandSolder
- J6: value SFH11-PBPC-D10-RA-BK -> SJ-3524-SMT; footprint connector:CONN20_D10-RA-BK_SUL -> Connector_Audio:Jack_3.5mm_CUI_SJ-3524-SMT_Horizontal
- Q3: value IRLML6402 -> MMBT2222A
- R4: value 5.1k -> 100k; footprint Capacitor_SMD:C_0603_1608Metric_Pad1.08x0.95mm_HandSolder -> Resistor_SMD:R_0603_1608Metric_Pad0.98x0.95mm_HandSolder
- U2: footprint RF_Module:ESP32-S3-WROOM-1U -> RF_Module:ESP32-S3-WROOM-1
- U6: value PCF8563T -> RT8059; footprint Package_SO:SOIC-8_3.9x4.9mm_P1.27mm -> Package_TO_SOT_SMD:TSOT-23-5_HandSoldering
- U7: value RT8059 -> TLV320AIC3100; footprint Package_TO_SOT_SMD:TSOT-23-5_HandSoldering -> Package_DFN_QFN:VQFN-32-1EP_5x5mm_P0.5mm_EP3.5x3.5mm
- U8: value TLV320AIC3100 -> PCF8563T; footprint Package_DFN_QFN:VQFN-32-1EP_5x5mm_P0.5mm_EP3.5x3.5mm -> Package_SO:SOIC-8_3.9x4.9mm_P1.27mm
- moved D2 177.7 mm to (382.7, 93.3)
- moved D4 136.2 mm to (382.7, 95.9)
- moved C1 127.5 mm to (363.5, 102.9)
- moved R4 112.9 mm to (367.8, 102.9)
- moved C2 107.8 mm to (363.5, 105.4)
- moved C13 106.4 mm to (358.3, 153.6)
- moved U6 88.0 mm to (282.0, 92.5)
- moved U8 86.8 mm to (273.8, 109.4)
- moved U7 83.3 mm to (226.0, 48.5)
- moved U4 56.5 mm to (281.1, 87.9)
- moved Q1 54.8 mm to (267.1, 108.5)
- moved TH1 52.0 mm to (231.5, 87.0), turned to 90 degrees
- moved Q2 47.3 mm to (233.1, 81.5)
- moved L1 46.8 mm to (281.8, 77.5)
- moved U1 35.7 mm to (215.0, 95.5)
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Connections:
- C1 pad 1: +VSW -> Net-(CHRG_VBUS1-B)
- C13 pad 1: +3.3V -> GND
- C13 pad 2: GND -> +BATT
- C2 pad 1: +3.3V -> +BATT
- C2 pad 2: Net-(U7-FB) -> GND
- D2 pad 1: Net-(D2-K) -> GND
- D2 pad 2: Net-(D2-A) -> Net-(D2-A2)
- D4 pad 1: PWRBTN_DETECT -> GND
- D4 pad 2: Net-(Q3-G) -> USB_DP
- J6 pad 2: Net-(F3-Pad2) -> GND
- J6 pad 3: OUT_RXD -> Net-(C21-Pad2)
- J6 pad 4: OUT_TXD -> Net-(U7-VOL/MICDET)
- L1 pad 1: Net-(U7-LX) -> Net-(U6-LX)
- L1 pad 2: +3.3V -> Net-(BUCK_POST1-B)
- Q1 pad 3: Net-(D2-A) -> Net-(D6-A)
- Q3 pad 1: Net-(Q3-G) -> Net-(Q3-B)
- Q3 pad 2: +BATT -> GND
- Q3 pad 3: +VSW -> Net-(J7-Pin_11)
- U1 pad 14: GND -> MCP_RESET
- U1 pad 15: MCP_INT_B -> unconnected-(U1-INTB-Pad15)
- U1 pad 16: unconnected-(U1-INTA-Pad16) -> MCP_INT
- U1 pad 24: unconnected-(U1-GPA7-Pad24) -> Net-(U1-GPA7)
- U2 pad 10: AUD_RESET -> TX_SIM_3V3
- U2 pad 11: AUD_DIN -> RX_SIM_3V3
- U2 pad 12: VIBRO_PIN -> MISO
- U2 pad 15: OUT_SCK -> SDA
- U2 pad 16: BOOT46 -> unconnected-(U2-IO46-Pad16)
- U2 pad 17: SDA -> MOSI
- U2 pad 18: SCK -> TF_CS
- U2 pad 19: CHG_PIN -> INT_ALARM
- U2 pad 20: PWR_HOLD -> MCP_RESET
- U2 pad 21: PWRBTN_DETECT -> MCP_INT
- U2 pad 22: SIM_RX -> PWRBTN_DETECT
- U2 pad 23: AUD_DOUT -> TF_DET
- U2 pad 24: IO47 -> AUD_DIN
- U2 pad 25: IO48 -> AUD_RESET
- U2 pad 26: MCP_INT_B -> unconnected-(U2-IO45-Pad26)
- U2 pad 27: BOOT0 -> SOC_BOOT
- U2 pad 28: OUT_IO_35 -> unconnected-(U2-IO35-Pad28)
- U2 pad 29: OUT_IO_36 -> unconnected-(U2-IO36-Pad29)
- U2 pad 3: ESP_EN -> SOC_EN
- U2 pad 30: OUT_IO_37 -> unconnected-(U2-IO37-Pad30)
- U2 pad 31: AUD_BCLK -> AUD_GPIO
- U2 pad 32: AUD_WCLK -> AUD_MCLK
- U2 pad 33: AUD_MCLK -> AUD_WCLK
- U2 pad 34: AUD_GPIO -> AUD_BCLK
- U2 pad 35: RTC_ALARM_INT -> AUD_DOUT
- U2 pad 36: OUT_RXD -> Net-(U2-RXD0)
- U2 pad 37: OUT_TXD -> Net-(U2-TXD0)
- U2 pad 38: OUT_MOSI -> SCK
- U2 pad 39: SD_CS -> VIB_CTRL
- U2 pad 4: OUT_MISO -> SCR_BL
- U2 pad 6: SD_DET -> DATA/COMMAND
- U2 pad 7: SCR_PWM -> SPI_CLOCK
- U2 pad 8: SIM_TX -> PWR_HOLD
- U2 pad 9: SIM_RI -> RI_SIM_3V3
- U4 pad 6: USB_VBUS -> Net-(CHRG_VBUS1-B)
- U6 pad 2: Net-(U6-OSCO) -> GND
- U6 pad 3: RTC_ALARM_INT -> Net-(U6-LX)
- U6 pad 4: GND -> Net-(BUCK_BAT1-A)
- U6 pad 5: SDA -> Net-(U6-FB)
- U7 pad 1: +VSW -> GND
- U7 pad 2: GND -> +3.3V
- U7 pad 3: Net-(U7-LX) -> +1V8
- U7 pad 4: +VSW -> AUD_DOUT
- U7 pad 5: Net-(U7-FB) -> AUD_DIN
- U8 pad 1: GND -> unconnected-(U8-OSCI-Pad1)
- U8 pad 2: +3.3V -> unconnected-(U8-OSCO-Pad2)
- U8 pad 3: +1V8 -> INT_ALARM
- U8 pad 4: AUD_DOUT -> GND
- U8 pad 5: AUD_DIN -> SDA
- U8 pad 6: AUD_WCLK -> SCK
- U8 pad 7: AUD_BCLK -> unconnected-(U8-CLKO-Pad7)
- U8 pad 8: AUD_MCLK -> +BATT

Commit message: lol
Parts:
- added ANT_GND1: SolderJumper_2_Open, Jumper:SolderJumper-2_P1.3mm_Open_Pad1.0x1.5mm, F.Cu at (273.2, 124.2)
- added C47: C, Capacitor_SMD:C_0603_1608Metric_Pad1.08x0.95mm_HandSolder, F.Cu at (268.8, 123.7)
- added C48: C, Capacitor_SMD:C_0603_1608Metric_Pad1.08x0.95mm_HandSolder, F.Cu at (268.8, 126.2)
- added J8: CONMHF4-SMD-G-T, CONMHF4-SMD-G-T:TE_CONMHF4-SMD-G-T, F.Cu at (273.0, 128.0)
- added R39: R, Resistor_SMD:R_0603_1608Metric_Pad0.98x0.95mm_HandSolder, F.Cu at (268.8, 128.7)
- added R40: R, Resistor_SMD:R_0603_1608Metric_Pad0.98x0.95mm_HandSolder, F.Cu at (268.8, 131.2)
- EAR_N1, EAR_P1, J1, J2, J4, MIC_N1, MIC_P1, SW_RST1, U2, U9: moved to B.Cu
- moved MIC_P1 185.7 mm to (190.0, 53.0), turned to 180 degrees
- moved MIC_N1 180.7 mm to (190.0, 57.0), turned to 180 degrees
- moved F1 179.0 mm to (199.6, 133.0), turned to 180 degrees
- moved EAR_P1 177.2 mm to (195.0, 53.0), turned to 180 degrees
- moved EAR_N1 173.8 mm to (193.0, 57.0), turned to 180 degrees
- moved SW_RST1 149.0 mm to (191.0, 134.0), turned to 180 degrees
- moved J1 147.2 mm to (204.0, 117.5), turned to -90 degrees
- moved J4 136.7 mm to (203.5, 101.6), turned to -90 degrees
- moved SW8 133.4 mm to (185.9, 104.8)
- moved J2 131.3 mm to (203.0, 85.5), turned to -90 degrees
- moved SW_BOOT1 114.5 mm to (225.6, 78.0)
- moved SW2 114.1 mm to (196.0, 89.6)
- moved SW10 109.5 mm to (209.6, 101.6)
- moved SW11 109.5 mm to (209.6, 108.0)
- moved SW12 109.5 mm to (209.6, 114.3)
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Connections:
- J5 pad A12_B1: (no net) -> GND
- J5 pad A4_B9: (no net) -> Net-(D2-A2)
- J5 pad B12_A1: (no net) -> GND
- J5 pad B4_A9: (no net) -> Net-(D2-A2)
- J5 pad SH1: (no net) -> GND
- J5 pad SH2: (no net) -> GND
- J6 pad 1: Net-(C20-Pad2) -> GND
- J6 pad 2: GND -> Net-(C20-Pad2)
- J6 pad 4: Net-(U7-VOL/MICDET) -> unconnected-(J6-Pad4)
- R6 pad 2: Net-(J5-CC1) -> Net-(J5-CC2)
- R7 pad 2: Net-(J5-CC2) -> Net-(J5-CC1)
- U7 pad 11: Net-(U7-VOL/MICDET) -> unconnected-(U7-VOL/MICDET-Pad11)
- U9 pad 60: unconnected-(U9-RF_ANT-Pad60) -> Net-(U9-RF_ANT)

Commit message: pcb progress
Parts:
- C14, C15, C16, C17, C18, C40, C41, C42, C43, C44, C45, C46, C7, R13, R14, R18, R19, R20, R21, R22, R33, R34, R35, R36, TP1, TP2, TP3, TP4, TP5, U10, U5: moved to B.Cu
- moved TXD1 193.4 mm to (197.0, 20.0), turned to -90 degrees
- moved TP9 193.0 mm to (195.0, 20.0), turned to -90 degrees
- moved TP8 186.4 mm to (201.0, 20.0), turned to -90 degrees
- moved RXD1 186.0 mm to (199.0, 20.0), turned to -90 degrees
- moved C45 174.9 mm to (169.0, 78.0), turned to -90 degrees
- moved U10 170.5 mm to (187.7, 85.8), turned to -90 degrees
- moved C46 167.8 mm to (176.6, 73.0), turned to 180 degrees
- moved R18 164.6 mm to (179.5, 82.0), turned to -90 degrees
- moved R19 164.5 mm to (181.7, 81.6), turned to -90 degrees
- moved U5 158.8 mm to (188.4, 104.5), turned to -90 degrees
- moved R36 158.4 mm to (193.2, 84.8)
- moved R35 155.8 mm to (193.3, 86.4)
- moved D2 155.6 mm to (231.0, 128.0)
- moved C44 153.0 mm to (193.0, 80.1), turned to 180 degrees
- moved R34 151.9 mm to (193.0, 91.3)
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
Commit message: P
Parts:
- removed SW20: POWER_BUTTON, PTS526_SM08_SMTR2_LFS:SW_PTS526_SM08_SMTR2_LFS
- added PCM_CLK1: TestPoint, TestPoint:TestPoint_Pad_D1.0mm, F.Cu at (1.02, 1.02)
- added PCM_DI1: TestPoint, TestPoint:TestPoint_Pad_D1.0mm, F.Cu at (1.02, 4.08)
- added PCM_DO1: TestPoint, TestPoint:TestPoint_Pad_D1.0mm, F.Cu at (1.02, 7.12)
- added PCM_S1: TestPoint, TestPoint:TestPoint_Pad_D1.0mm, F.Cu at (1.02, 10.2)
- added SW24: SW_MEC_5E, PTS526_SM08_SMTR2_LFS:SW_PTS526_SM08_SMTR2_LFS, F.Cu at (9.65, 2.67)
- J1: value Micro_SD_Card_Det1 -> DM3D-SF; footprint Connector_Card:microSD_HC_Hirose_DM3AT-SF-PEJM5 -> DM3D-SF:HRS_DM3D-SF
Connections:
- J2 pad SH: (no net) -> GND
- J3 pad 0: (no net) -> unconnected-(J3-NC-Pad0)_2
- J4 pad SH: (no net) -> GND
- U9 pad 11: unconnected-(U9-PCM_CLK-Pad11) -> Net-(U9-PCM_CLK)
- U9 pad 12: unconnected-(U9-PCM_SYNC-Pad12) -> Net-(U9-PCM_SYNC)
- U9 pad 13: unconnected-(U9-PCM_DIN-Pad13) -> Net-(U9-PCM_DIN)
- U9 pad 14: unconnected-(U9-PCM_DOUT-Pad14) -> Net-(U9-PCM_DOUT)
