File: power.kicad_sch (KiCad schematic)
At the start: 33 parts, among them J3 BATTERY, J5 USB_C_Receptacle_USB2.0_16P, SW20 POWER_BUTTON, U4 BQ21040DBV, U6 RT8059

Commit message: lol
Parts:
- J5: symbol Connector:USB_C_Receptacle_USB2.0_16P -> UJ20-C-G-MSMT-TR-68:UJ20-C-G-MSMT-TR-68; MANUFACTURER (none) -> CUI Devices; PARTREV (none) -> 1.0; STANDARD (none) -> Manufacturer Recommendations
Connections:
- net GND: now also J5.A12_B1 (GND), J5.B12_A1 (GND__1), J5.SH1 (SHIELD), J5.SH2 (SHIELD__1); no longer J5.A1 (GND), J5.A12 (GND), J5.B1 (GND), J5.B12 (GND), J5.S1 (SHIELD)
- net at R6.2: now also J5.B5 (CC2); no longer J5.A5 (CC1)
- net at R7.2: now also J5.A5 (CC1); no longer J5.B5 (CC2)
- new net: D2.2 (A2), F1.1, J5.A4_B9 (VBUS), J5.B4_A9 (VBUS__1)
Other:
- moved on the sheet: D2, D4, D5, R4, R6, R7, R8

Commit message: what
Parts:
- removed SW20: POWER_BUTTON, PTS526_SM08_SMTR2_LFS:SW_PTS526_SM08_SMTR2_LFS, symbol Switch:SW_Push
- added SW24: SW_MEC_5E, PTS526_SM08_SMTR2_LFS:SW_PTS526_SM08_SMTR2_LFS, symbol Switch:SW_MEC_5E
Connections:
- net GND: now also SW24.1, SW24.2
- net at D1.3 (K): now also SW24.3 (K), SW24.4 (A)
Changed lines of the file:
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@@
 	)
 	(junction
+		(at 57.15 57.15)
+		(diameter 0)
+		(color 0 0 0 0)
+	)
+	(junction
 		(at 55.88 74.93)
 		(diameter 0)
@@
 	)
 	(junction
+		(at 46.99 57.15)
+		(diameter 0)
+		(color 0 0 0 0)
+	)
+	(junction
 		(at 36.83 140.97)
 		(diameter 0)
@@
 	(wire
 		(pts
+			(xy 46.99 54.61) (xy 46.99 57.15)
+		)
+		(stroke
+			(width 0)
+			(type default)
+		)
+	)
+	(wire
+		(pts
 			(xy 64.77 177.8) (xy 64.77 171.45)
 		)
@@
 	(wire
 		(pts
+			(xy 57.15 54.61) (xy 57.15 57.15)
+		)
+		(stroke
+			(width 0)
+			(type default)
+		)
+	)
+	(wire
+		(pts
 			(xy 54.61 88.9) (xy 54.61 81.28)
 		)
@@
 	)
 	(symbol
-		(lib_id "Switch:SW_Push")
-		(at 52.07 57.15 0)
-		(unit 1)
-		(exclude_from_sim no)
-		(in_bom yes)
-		(on_board yes)
-		(dnp no)
-		(property "Reference" "SW20"
-			(at 52.07 49.53 0)
-			(effects
-				(font
-					(size 1.27 1.27)
-				)
-			)
-		)
-		(property "Value" "POWER_BUTTON"
-			(at 48.006 51.816 0)
-			(effects
-				(font
-					(size 1.27 1.27)
-				)
-			)
-		)
-		(property "Footprint" "PTS526_SM08_SMTR2_LFS:SW_PTS526_SM08_SMTR2_LFS"
-			(at 52.07 52.07 0)
-			(effects
-				(font
-					(size 1.27 1.27)
-				)
-				(hide yes)
-			)
-		)
-		(property "Datasheet" "~"
-			(at 52.07 52.07 0)
-			(effects
-				(font
-					(size 1.27 1.27)
-				)
-				(hide yes)
-			)
-		)
-		(property "Description" "Push button switch, generic, two pins"
-			(at 52.07 57.15 0)
-			(effects
-				(font
-					(size 1.27 1.27)
-				)
-				(hide yes)
-			)
-		)
-		(pin "1"
-		)
-		(pin "2"
-		)
-		(instances
-			(project "power"
-				(path "/b8244a46-7ec4-4641-80d4-82c2f8ffc6ae"
-					(reference "SW?")
-					(unit 1)
-				)
-			)
-			(project "power"
-				(path "/e9d3405d-3536-4ebc-8db6-e75908125fac/4fc341b7-aab9-4bf1-942c-802f704f4f3e"
-					(reference "SW20")
-					(unit 1)
-				)
-			)
-		)
-	)
-	(symbol
 		(lib_id "power:GND")
 		(at 152.4 100.33 0)
@@
 					(unit 1)
 				)
+			)
+		)
+	)
+	(symbol
+		(lib_id "Switch:SW_MEC_5E")
+		(at 52.07 57.15 0)
+		(unit 1)
+		(exclude_from_sim no)
+		(in_bom yes)
+		(on_board yes)
+		(dnp no)
+		(property "Reference" "SW24"
+			(at 52.07 56.642 0)
+			(effects
+				(font
+					(size 1.27 1.27)
+				)
+			)
+		)
+		(property "Value" "SW_MEC_5E"
+			(at 52.07 49.53 0)
+			(effects
+				(font
+					(size 1.27 1.27)
+				)
+				(hide yes)
+			)
+		)
+		(property "Footprint" "PTS526_SM08_SMTR2_LFS:SW_PTS526_SM08_SMTR2_LFS"
+			(at 52.07 49.53 0)
+			(effects
+				(font
+					(size 1.27 1.27)
+				)
+				(hide yes)
+			)
+		)
+		(property "Datasheet" "http://www.apem.com/int/index.php?controller=attachment&id_attachment=1371"
+			(at 52.07 49.53 0)
+			(effects
+				(font
+					(size 1.27 1.27)
+				)
+				(hide yes)
+			)
+		)
+		(property "Description" "MEC 5E single pole normally-open tactile switch"
+			(at 52.07 57.15 0)
+			(effects
+				(font
+					(size 1.27 1.27)
+				)
+				(hide yes)
+			)
+		)
+		(pin "4"
+		)
+		(pin "3"
+		)
+		(pin "2"
+		)
+		(pin "1"
+		)
+		(instances
+			(project "okabephone"
+				(path "/e9d3405d-3536-4ebc-8db6-e75908125fac/4fc341b7-aab9-4bf1-942c-802f704f4f3e"
+					(reference "SW24")
+					(unit 1)
+				)

Commit message: P
Changed lines of the file:
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@@
 		(pin "1"
+		)
+		(pin "0"
 		)
 		(instances
